File: EAGLE Models/BMS/BMS(board layout version).brd (EAGLE design)
At the start: 160 x 100 mm, 25 parts

Commit message: Cleaned up Schematic
Connections:
- net GATE renamed N$10
- net POS renamed N$13
Changed lines of the file:
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@@
 <signals>
 <signal name="VCC">
+<contactref element="U$4" pad="P$1"/>
 <contactref element="R7" pad="2"/>
-<contactref element="C1" pad="1"/>
 <contactref element="R1" pad="2"/>
-<contactref element="R6" pad="2"/>
+<contactref element="U$4" pad="P$2"/>
 <contactref element="R11" pad="2"/>
 <contactref element="U$5" pad="P$8"/>
-<contactref element="U$4" pad="P$1"/>
-<contactref element="U$4" pad="P$2"/>
+<contactref element="R6" pad="2"/>
+<contactref element="C1" pad="1"/>
 <wire x1="48.26" y1="46.67" x2="66.99" y2="49.53" width="0" layer="19" extent="1-1"/>
 <wire x1="44.45" y1="40.96" x2="48.26" y2="46.67" width="0" layer="19" extent="1-1"/>
@@
 <wire x1="33.34" y1="38.37" x2="34.29" y2="40.37" width="0" layer="19" extent="1-1"/>
 <wire x1="23.81" y1="33.02" x2="33.34" y2="38.37" width="0" layer="19" extent="1-1"/>
+<wire x1="39.65" y1="22.5815" x2="33.34" y2="38.37" width="0" layer="19" extent="1-1"/>
 <wire x1="11.75" y1="25.4" x2="23.81" y2="33.02" width="0" layer="19" extent="1-1"/>
-<wire x1="39.65" y1="22.5815" x2="33.34" y2="38.37" width="0" layer="19" extent="1-1"/>
 </signal>
 <signal name="N$4">
@@
 <signal name="GND">
 <contactref element="U$2" pad="P$4"/>
+<contactref element="U$1" pad="P$4"/>
 <contactref element="U$5" pad="P$4"/>
+<contactref element="R8" pad="1"/>
+<contactref element="LED1" pad="C"/>
+<contactref element="LED2" pad="A"/>
 <contactref element="U$3" pad="P$3"/>
+<contactref element="U$4" pad="P$3"/>
+<contactref element="C2" pad="2"/>
+<contactref element="C1" pad="2"/>
 <contactref element="NEG" pad="1"/>
-<contactref element="C2" pad="2"/>
-<contactref element="U$4" pad="P$3"/>
-<contactref element="C1" pad="2"/>
-<contactref element="LED2" pad="A"/>
-<contactref element="LED1" pad="C"/>
-<contactref element="R8" pad="1"/>
-<contactref element="U$1" pad="P$4"/>
 <wire x1="82.87" y1="27.94" x2="73.571" y2="47.31" width="0" layer="19" extent="1-1"/>
 <wire x1="56.83" y1="12.97" x2="82.87" y2="27.94" width="0" layer="19" extent="1-1"/>
@@
 </signal>
 <signal name="DOWN">
+<contactref element="DOWN" pad="1"/>
 <contactref element="R2" pad="2"/>
 <contactref element="R1" pad="1"/>
-<contactref element="DOWN" pad="1"/>
 <wire x1="55.88" y1="33.34" x2="50.8" y2="64.77" width="0" layer="19" extent="1-1"/>
 <wire x1="21.91" y1="33.02" x2="55.88" y2="33.34" width="0" layer="19" extent="1-1"/>
@@
 <wire x1="71.209" y1="47.31" x2="31.43" y2="29.21" width="0" layer="19" extent="1-1"/>
 </signal>
+<signal name="N$16">
+<contactref element="U$5" pad="P$1"/>
+<contactref element="R11" pad="1"/>
+<wire x1="48.26" y1="44.77" x2="34.01" y2="22.5815" width="0" layer="19" extent="1-1"/>
+</signal>
 <signal name="N$6">
 <contactref element="R2" pad="1"/>
@@
 <wire x1="55.88" y1="35.24" x2="39.65" y2="20.5985" width="0" layer="19" extent="1-1"/>
 </signal>
-<signal name="POS">
+<signal name="N$13">
 <contactref element="POS" pad="1"/>
 <contactref element="R12" pad="1"/>
@@
 <wire x1="39.65" y1="21.2595" x2="54.93" y2="12.97" width="0" layer="19" extent="1-1"/>
 </signal>
+<signal name="N$8">
+<contactref element="U$2" pad="P$8"/>
+<contactref element="R6" pad="1"/>
+<contactref element="R5" pad="1"/>
+<contactref element="C2" pad="1"/>
+<wire x1="44.45" y1="42.86" x2="78.74" y2="15.56" width="0" layer="19" extent="1-1"/>
+<wire x1="23.02" y1="51.435" x2="44.45" y2="42.86" width="0" layer="19" extent="1-1"/>
+<wire x1="7.94" y1="20.32" x2="23.02" y2="51.435" width="0" layer="19" extent="1-1"/>
+</signal>
 <signal name="N$7">
 <contactref element="U$5" pad="P$2"/>
@@
 <wire x1="34.01" y1="21.9205" x2="78.74" y2="17.46" width="0" layer="19" extent="1-1"/>
 </signal>
-<signal name="GATE">
+<signal name="N$10">
+<contactref element="U$5" pad="P$3"/>
 <contactref element="R4" pad="1"/>
 <contactref element="R8" pad="2"/>
 <contactref element="R9" pad="2"/>
-<contactref element="U$5" pad="P$3"/>
 <wire x1="84.77" y1="27.94" x2="97.47" y2="29.21" width="0" layer="19" extent="1-1"/>
 <wire x1="34.01" y1="21.2595" x2="84.77" y2="27.94" width="0" layer="19" extent="1-1"/>
@@
 <wire x1="31.75" y1="46.51" x2="82.87" y2="41.91" width="0" layer="19" extent="1-1"/>
 </signal>
-<signal name="N$1">
-<contactref element="U$2" pad="P$8"/>
-<contactref element="R6" pad="1"/>
-<contactref element="R5" pad="1"/>
-<contactref element="C2" pad="1"/>
-<wire x1="44.45" y1="42.86" x2="78.74" y2="15.56" width="0" layer="19" extent="1-1"/>
-<wire x1="23.02" y1="51.435" x2="44.45" y2="42.86" width="0" layer="19" extent="1-1"/>
-<wire x1="7.94" y1="20.32" x2="23.02" y2="51.435" width="0" layer="19" extent="1-1"/>
-</signal>
-<signal name="N$2">
+<signal name="N$14">
 <contactref element="U$5" pad="P$7"/>
 <contactref element="R10" pad="2"/>
 <wire x1="39.65" y1="21.9206" x2="84.77" y2="41.91" width="0" layer="19" extent="1-1"/>
 </signal>
-<signal name="N$5">
-<contactref element="U$5" pad="P$1"/>
-<contactref element="R11" pad="1"/>
-<wire x1="34.01" y1="22.5815" x2="48.26" y2="44.77" width="0" layer="19" extent="1-1"/>
-</signal>
 </signals>
