File: EAGLE Models/BMS/BMS Rev. 1.brd (EAGLE design)
At the start: 160 x 100 mm, 25 parts

Commit message: Started schematic of temperature measurement circuit
Parts:
- C1: value (none) -> 15uF??
- C2: value (none) -> 10-40uF
Connections:
- removed net N$12: LED2.C, R10.1
- new net N$8: LED2.A, R10.1
- net GND: now also LED2.C; no longer LED2.A
Changed lines of the file:
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@@
 <element name="POS" library="formula electric" package="CONNECTOR_1" value="CONN_1" x="40.64" y="66.04"/>
 <element name="NEG" library="formula electric" package="CONNECTOR_1" value="CONN_1" x="10.16" y="52.07"/>
-<element name="C2" library="resistor" package="C0805" value="" x="8.89" y="20.32"/>
-<element name="C1" library="resistor" package="C0805" value="" x="12.7" y="25.4"/>
+<element name="C2" library="resistor" package="C0805" value="10-40uF" x="8.89" y="20.32"/>
+<element name="C1" library="resistor" package="C0805" value="15uF??" x="12.7" y="25.4"/>
 </elements>
 <signals>
@@
 <contactref element="U$4" pad="P$3"/>
 <contactref element="C1" pad="2"/>
-<contactref element="LED2" pad="A"/>
 <contactref element="LED1" pad="C"/>
 <contactref element="R8" pad="1"/>
@@
 <contactref element="U$5" pad="P$4"/>
 <contactref element="U$2" pad="P$4"/>
+<contactref element="LED2" pad="C"/>
 <wire x1="82.87" y1="27.94" x2="73.571" y2="47.31" width="0" layer="19" extent="1-1"/>
 <wire x1="56.83" y1="12.97" x2="82.87" y2="27.94" width="0" layer="19" extent="1-1"/>
 <wire x1="34.01" y1="20.5985" x2="56.83" y2="12.97" width="0" layer="19" extent="1-1"/>
 <wire x1="35.24" y1="38.37" x2="34.01" y2="20.5985" width="0" layer="19" extent="1-1"/>
-<wire x1="36.83" y1="50.01" x2="35.24" y2="38.37" width="0" layer="19" extent="1-1"/>
-<wire x1="31.75" y1="50.01" x2="36.83" y2="50.01" width="0" layer="19" extent="1-1"/>
-<wire x1="17.62" y1="47.625" x2="31.75" y2="50.01" width="0" layer="19" extent="1-1"/>
+<wire x1="31.75" y1="46.51" x2="35.24" y2="38.37" width="0" layer="19" extent="1-1"/>
+<wire x1="36.83" y1="50.01" x2="31.75" y2="46.51" width="0" layer="19" extent="1-1"/>
+<wire x1="17.62" y1="47.625" x2="31.75" y2="46.51" width="0" layer="19" extent="1-1"/>
 <wire x1="10.16" y1="52.07" x2="17.62" y2="47.625" width="0" layer="19" extent="1-1"/>
 <wire x1="13.65" y1="25.4" x2="34.01" y2="20.5985" width="0" layer="19" extent="1-1"/>
@@
 <wire x1="36.83" y1="46.51" x2="95.57" y2="29.21" width="0" layer="19" extent="1-1"/>
 </signal>
-<signal name="N$12">
-<contactref element="R10" pad="1"/>
-<contactref element="LED2" pad="C"/>
-<wire x1="31.75" y1="46.51" x2="82.87" y2="41.91" width="0" layer="19" extent="1-1"/>
-</signal>
 <signal name="N$1">
 <contactref element="U$2" pad="P$8"/>
@@
 <wire x1="34.01" y1="22.5815" x2="48.26" y2="44.77" width="0" layer="19" extent="1-1"/>
 </signal>
+<signal name="N$8">
+<contactref element="R10" pad="1"/>
+<contactref element="LED2" pad="A"/>
+<wire x1="31.75" y1="50.01" x2="82.87" y2="41.91" width="0" layer="19" extent="1-1"/>
+</signal>
 </signals>

Commit message: First board layout attempt
Parts:
- C1: value 15uF?? -> 17-20uF
- C2: value 10-40uF -> 100nF
Connections:
- net DOWN: now also DOWN.2
- net GND: now also NEG.2
- net POS: now also POS.2
- net UP: now also UP.2
Changed lines of the file:
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@@
 <element name="POS" library="formula electric" package="CONNECTOR_1" value="CONN_1" x="40.64" y="66.04"/>
 <element name="NEG" library="formula electric" package="CONNECTOR_1" value="CONN_1" x="10.16" y="52.07"/>
-<element name="C2" library="resistor" package="C0805" value="10-40uF" x="8.89" y="20.32"/>
-<element name="C1" library="resistor" package="C0805" value="15uF??" x="12.7" y="25.4"/>
+<element name="C2" library="resistor" package="C0805" value="100nF" x="8.89" y="20.32"/>
+<element name="C1" library="resistor" package="C0805" value="17-20uF" x="12.7" y="25.4"/>
 </elements>
 <signals>
@@
 <contactref element="U$2" pad="P$4"/>
 <contactref element="LED2" pad="C"/>
+<contactref element="NEG" pad="2"/>
 <wire x1="82.87" y1="27.94" x2="73.571" y2="47.31" width="0" layer="19" extent="1-1"/>
 <wire x1="56.83" y1="12.97" x2="82.87" y2="27.94" width="0" layer="19" extent="1-1"/>
@@
 <wire x1="17.62" y1="47.625" x2="31.75" y2="46.51" width="0" layer="19" extent="1-1"/>
 <wire x1="10.16" y1="52.07" x2="17.62" y2="47.625" width="0" layer="19" extent="1-1"/>
+<wire x1="12.66" y1="57.07" x2="10.16" y2="52.07" width="0" layer="19" extent="1-1"/>
 <wire x1="13.65" y1="25.4" x2="34.01" y2="20.5985" width="0" layer="19" extent="1-1"/>
 <wire x1="9.84" y1="20.32" x2="13.65" y2="25.4" width="0" layer="19" extent="1-1"/>
@@
 <contactref element="R1" pad="1"/>
 <contactref element="DOWN" pad="1"/>
+<contactref element="DOWN" pad="2"/>
+<wire x1="50.8" y1="64.77" x2="53.3" y2="69.77" width="0" layer="19" extent="1-1"/>
 <wire x1="55.88" y1="33.34" x2="50.8" y2="64.77" width="0" layer="19" extent="1-1"/>
 <wire x1="21.91" y1="33.02" x2="55.88" y2="33.34" width="0" layer="19" extent="1-1"/>
@@
 <contactref element="UP" pad="1"/>
 <contactref element="R3" pad="2"/>
+<contactref element="UP" pad="2"/>
+<wire x1="66.04" y1="66.04" x2="68.54" y2="71.04" width="0" layer="19" extent="1-1"/>
 <wire x1="55.88" y1="22.54" x2="66.04" y2="66.04" width="0" layer="19" extent="1-1"/>
 </signal>
@@
 <contactref element="R12" pad="1"/>
 <contactref element="R7" pad="1"/>
+<contactref element="POS" pad="2"/>
 <wire x1="65.09" y1="49.53" x2="70.17" y2="53.34" width="0" layer="19" extent="1-1"/>
 <wire x1="40.64" y1="66.04" x2="65.09" y2="49.53" width="0" layer="19" extent="1-1"/>
+<wire x1="43.14" y1="71.04" x2="40.64" y2="66.04" width="0" layer="19" extent="1-1"/>
 </signal>
 <signal name="N$9">
