File: EAGLE Models/BMS CAN/BMS Temp CAN Module.brd (EAGLE design)
At the start: 160 x 100 mm, 106 parts, among them IC1 AT90CAN128, IC2 MCP2551SO8, IC3 NUP2105L, IC5 FT232RL, Q1 56P2859, X1 AS16-35, X2 AS06-05, X3 MOLEX_CONN_20, X4 MOLEX_CONN_20, X5 MOLEX_CONN_20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

Commit message: Revert "Dont Remember"
This reverts commit 84a080d4c1201f3fd16338f4fffe7880c36af064.
Parts:
- removed X3, X4, X5, X6: MOLEX_CONN_20, BMS Temp CAN Board:WM7492
Connections:
- removed net A25: X4.P$4
- removed net A26: X4.P$14
- removed net A27: X4.P$5
- removed net A28: X4.P$15
- removed net A29: X4.P$6
- removed net A30: X4.P$16
- removed net A31: X4.P$7
- removed net A32: X4.P$17
- removed net A33: X4.P$8
- removed net A34: X4.P$18
- removed net A35: X4.P$9
- removed net A36: X4.P$19
- removed net A37: X5.P$1
- removed net A38: X5.P$11
- removed net A39: X5.P$2
- removed net A40: X5.P$12
- removed net A41: X5.P$3
- removed net A42: X5.P$13
- removed net A43: X5.P$4
- removed net A44: X5.P$14
- removed net A45: X5.P$5
- removed net A46: X5.P$15
- removed net A47: X5.P$6
- removed net A48: X5.P$16
- removed net A49: X5.P$7
- removed net A50: X5.P$17
- removed net A51: X5.P$8
- removed net A52: X5.P$18
- removed net A53: X5.P$9
- removed net A54: X5.P$19
- removed net A55: X6.P$1
- removed net A56: X6.P$11
- removed net A57: X6.P$2
- removed net A58: X6.P$12
- removed net A59: X6.P$3
- removed net A60: X6.P$13
- removed net A61: X6.P$4
- removed net A62: X6.P$14
- removed net A63: X6.P$5
- removed net A64: X6.P$15
- removed net A65: X6.P$6
- removed net A66: X6.P$16
- removed net A67: X6.P$7
- removed net A68: X6.P$17
- removed net A69: X6.P$8
- removed net A70: X6.P$18
- removed net A71: X6.P$9
- removed net A72: X6.P$19
- net A1: no longer X3.P$1
- net A10: no longer X3.P$15
- net A11: no longer X3.P$6
- net A12: no longer X3.P$16
- net A13: no longer X3.P$7
- net A14: no longer X3.P$17
- net A15: no longer X3.P$8
- net A16: no longer X3.P$18
- net A17: no longer X3.P$9
- net A18: no longer X3.P$19
- net A19: no longer X4.P$1
- net A2: no longer X3.P$11
- net A20: no longer X4.P$11
- net A21: no longer X4.P$2
- net A22: no longer X4.P$12
- net A23: no longer X4.P$3
- net A24: no longer X4.P$13
- net A3: no longer X3.P$2
- net A4: no longer X3.P$12
- net A5: no longer X3.P$3
- net A6: no longer X3.P$13
- net A7: no longer X3.P$4
- net A8: no longer X3.P$14
- net A9: no longer X3.P$5
- net GND: no longer X3.P$20, X4.P$20, X5.P$20, X6.P$20
- net VCC: no longer X3.P$10, X4.P$10, X5.P$10, X6.P$10
