File: EAGLE Models/BMS/BMS CAN/BMS Temp CAN Module.brd (EAGLE design)
At the start: 160 x 100 mm, 102 parts, among them IC1 AT90CAN128, IC2 MCP2551SO8, IC3 NUP2105L, IC5 FT232RL, Q1 56P2859, X1 AS16-35, X2 AS06-05

Commit message: Revert "Revert "Dont Remember""
This reverts commit 58ed382bf306966dc374cccd45e7e33cb299af38.
Parts:
- added X3, X4, X5, X6: MOLEX_CONN_20, BMS Temp CAN Board:WM7492
Connections:
- new net A25: X4.P$4
- new net A26: X4.P$14
- new net A27: X4.P$5
- new net A28: X4.P$15
- new net A29: X4.P$6
- new net A30: X4.P$16
- new net A31: X4.P$7
- new net A32: X4.P$17
- new net A33: X4.P$8
- new net A34: X4.P$18
- new net A35: X4.P$9
- new net A36: X4.P$19
- new net A37: X5.P$1
- new net A38: X5.P$11
- new net A39: X5.P$2
- new net A40: X5.P$12
- new net A41: X5.P$3
- new net A42: X5.P$13
- new net A43: X5.P$4
- new net A44: X5.P$14
- new net A45: X5.P$5
- new net A46: X5.P$15
- new net A47: X5.P$6
- new net A48: X5.P$16
- new net A49: X5.P$7
- new net A50: X5.P$17
- new net A51: X5.P$8
- new net A52: X5.P$18
- new net A53: X5.P$9
- new net A54: X5.P$19
- new net A55: X6.P$1
- new net A56: X6.P$11
- new net A57: X6.P$2
- new net A58: X6.P$12
- new net A59: X6.P$3
- new net A60: X6.P$13
- new net A61: X6.P$4
- new net A62: X6.P$14
- new net A63: X6.P$5
- new net A64: X6.P$15
- new net A65: X6.P$6
- new net A66: X6.P$16
- new net A67: X6.P$7
- new net A68: X6.P$17
- new net A69: X6.P$8
- new net A70: X6.P$18
- new net A71: X6.P$9
- new net A72: X6.P$19
- net A1: now also X3.P$1
- net A10: now also X3.P$15
- net A11: now also X3.P$6
- net A12: now also X3.P$16
- net A13: now also X3.P$7
- net A14: now also X3.P$17
- net A15: now also X3.P$8
- net A16: now also X3.P$18
- net A17: now also X3.P$9
- net A18: now also X3.P$19
- net A19: now also X4.P$1
- net A2: now also X3.P$11
- net A20: now also X4.P$11
- net A21: now also X4.P$2
- net A22: now also X4.P$12
- net A23: now also X4.P$3
- net A24: now also X4.P$13
- net A3: now also X3.P$2
- net A4: now also X3.P$12
- net A5: now also X3.P$3
- net A6: now also X3.P$13
- net A7: now also X3.P$4
- net A8: now also X3.P$14
- net A9: now also X3.P$5
- net GND: now also X3.P$20, X4.P$20, X5.P$20, X6.P$20
- net VCC: now also X3.P$10, X4.P$10, X5.P$10, X6.P$10
