File: EAGLE Models/BMS/ADC Boards/ADC Board(Two Board,Molex).sch (EAGLE design)
At the start: 35 parts, among them IC1 ADS7956, IC2 ADS7956, IC3 ADS7956, X1 6_PIN_CONNMOLEX_HORI, X10 6_PIN_CONNMOLEX_HORI, X2 6_PIN_CONNMOLEX_HORI, X3 6_PIN_CONNMOLEX_HORI, X4 6_PIN_CONNMOLEX_HORI, X5 6_PIN_CONNMOLEX_HORI, X6 6_PIN_CONNMOLEX_HORI, X7 8_PIN_CONN, X8 6_PIN_CONNMOLEX_HORI, X9 6_PIN_CONNMOLEX_HORI

Commit message: CAN Board Layout
Parts:
- added C13, C14: .1uF, rcl:C-EUC0603
- added R4, R5: 100k, rcl:R-US_M0805
Connections:
- removed net N$1: U$2.VIN
- removed net N$2: U$2.GND
- removed net N$4: U$2.EN
- removed net N$5: U$2.VOUT
- removed net VA: C1.1, C11.1, C3.1, C5.1, C7.1, C9.1, IC1.+VA1, IC1.+VA2, IC2.+VA1, IC2.+VA2, IC3.+VA1, IC3.+VA2, X1/2.$/1, X10/2.$/1, X2/2.$/1, X3/2.$/1, X4/2.$/1, X5/2.$/1, X6/2.$/1, X8/2.$/1, X9/2.$/1
- new net 12V: C14.1, R4.2, U$2.VIN, X7/2.$/1
- new net ENABLE: R4.1, R5.2, U$2.EN
- net GND: now also C13.2, C14.2, R5.1, U$2.GND
- net VCC: now also C1.1, C11.1, C13.1, C3.1, C5.1, C7.1, C9.1, IC1.+VA1, IC1.+VA2, IC2.+VA1, IC2.+VA2, IC3.+VA1, IC3.+VA2, U$2.VOUT, X1/2.$/1, X10/2.$/1, X2/2.$/1, X3/2.$/1, X4/2.$/1, X5/2.$/1, X6/2.$/1, X8/2.$/1, X9/2.$/1; no longer X7/2.$/1

Commit message: Moved things
Other:
- note added: "5V Supply"
- moved on the sheet: X1/1, X1/2, X1/3, X1/4, X1/5, X1/6, X10/1, X10/2, X10/3, X10/4, X10/5, X10/6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
