File: EAGLE Models/BMS/BMS MiniCAN Boards/BMS MiniCAN Board Thermistor Wires.brd (EAGLE design)
At the start: 102.8 x 59.4 mm, 74 parts, among them IC1 AT90CAN128, IC2 MCP2551SO8, IC3 NUP2105L, IC5 FT232RL, Q1 56P2859, X2 6_PIN_CONNMOLEX_HORI, X3 6_PIN_CONNMOLEX_HORI, X4 6_PIN_CONNMOLEX_HORI, X5 6_PIN_CONNMOLEX_HORI, X6 6_PIN_CONNMOLEX_HORI

Commit message: Connected thermistor connectors and general cleanup
Connected the thermistor connectors to the muxes and fixed some issues
with the connector itself. Also deleted the old ADC.
Parts:
- removed C5, C6: .1uF, rcl:C0805
- removed C7, C8: 1uF, rcl:C0805
- removed R4: 51, adafruit:R0805
- removed U$2: ADC084S101, BMS Lbr:TSSOP-16
- removed X2, X3, X4, X5, X6: 6_PIN_CONNMOLEX_HORI, BMS Lbr:6_PIN_MOLEX
- added U$10, U$11, U$12, U$13, U$3, U$9: 10127720-241LF, con-amphenol:10127720-241LF
Connections:
- removed net NC: X2.P$3
- removed net NC1: X3.P$3
- removed net NC2: X4.P$3
- removed net NC3: X5.P$3
- removed net NC4: X6.P$3
- removed net VD: C6.1, C8.1, R4.2, U$2.P$13
- new net AIN72: U$11.P$24
- net AIN0: now also U$12.P$13; no longer X2.P$4
- net AIN1: now also U$12.P$14; no longer X2.P$5
- net AIN10: now also U$12.P$23; no longer U$2.P$8, X5.P$5
- net AIN11: no longer U$2.P$7, X5.P$6
- net AIN12: now also U$12.P$24; no longer U$2.P$6, X6.P$4
- net AIN13: now also U$13.P$13; no longer U$2.P$5, X6.P$5
- net AIN14: now also U$13.P$14; no longer U$2.P$4, X6.P$6
- net AIN15: now also U$13.P$15
- net AIN16: now also U$13.P$16
- net AIN17: now also U$13.P$17
- net AIN18: now also U$13.P$18
- net AIN19: now also U$13.P$19
- net AIN2: now also U$12.P$15; no longer X2.P$6
- net AIN20: now also U$13.P$20
- net AIN21: now also U$13.P$21
- net AIN22: now also U$13.P$22
- net AIN23: now also U$13.P$23
- net AIN24: now also U$13.P$24
- net AIN25: now also U$3.P$13
- net AIN26: now also U$3.P$14
- net AIN27: now also U$3.P$15
- net AIN28: now also U$3.P$16
- net AIN29: now also U$3.P$17
- net AIN3: now also U$12.P$16; no longer X3.P$4
- net AIN30: now also U$3.P$18
- net AIN31: now also U$3.P$19
- net AIN32: now also U$3.P$20
- net AIN33: now also U$3.P$21
- net AIN34: now also U$3.P$22
- net AIN35: now also U$3.P$23
- net AIN36: now also U$3.P$24
- net AIN37: now also U$9.P$13
- net AIN38: now also U$9.P$14
- net AIN39: now also U$9.P$15
- net AIN4: now also U$12.P$17; no longer X3.P$5
- net AIN40: now also U$9.P$16
- net AIN41: now also U$9.P$17
- net AIN42: now also U$9.P$18
- net AIN43: now also U$9.P$19
- net AIN44: now also U$9.P$20
- net AIN45: now also U$9.P$21
- net AIN46: now also U$9.P$22
- net AIN47: now also U$9.P$23
- net AIN48: now also U$9.P$24
- net AIN49: now also U$10.P$13
- net AIN5: now also U$12.P$18; no longer X3.P$6
- net AIN50: now also U$10.P$14
- net AIN51: now also U$10.P$15
- net AIN52: now also U$10.P$16
- net AIN53: now also U$10.P$17
- net AIN54: now also U$10.P$18
- net AIN55: now also U$10.P$19
- net AIN56: now also U$10.P$20
- net AIN57: now also U$10.P$21
- net AIN58: now also U$10.P$22
- net AIN59: now also U$10.P$23
- net AIN6: now also U$12.P$19; no longer X4.P$4
- net AIN60: now also U$10.P$24
- net AIN61: now also U$11.P$13
- net AIN62: now also U$11.P$14
- net AIN63: now also U$11.P$15
- net AIN64: now also U$11.P$16
- net AIN65: now also U$11.P$17
- net AIN66: now also U$11.P$18
- net AIN67: now also U$11.P$19
- net AIN68: now also U$11.P$20
- net AIN69: now also U$11.P$21
- net AIN7: now also U$12.P$20; no longer X4.P$5
- net AIN70: now also U$11.P$22
- net AIN71: now also U$11.P$23
- net AIN8: now also U$12.P$21; no longer U$2.P$10, X4.P$6
- net AIN9: now also U$12.P$22; no longer U$2.P$9, X5.P$4
- net CS: no longer U$2.P$1
- net DIN: no longer U$2.P$14
- net DOUT: no longer U$2.P$15
- net GND: no longer C5.2, C6.2, C7.2, C8.2, U$2.P$11, U$2.P$12, U$2.P$3, X2.P$1, X3.P$1, X4.P$1, X5.P$1, X6.P$1
- net SCLK: no longer U$2.P$16
- net VCC: now also U$10.P$1, U$10.P$10, U$10.P$11, U$10.P$12, U$10.P$2, U$10.P$3, U$10.P$4, U$10.P$5, U$10.P$6, U$10.P$7, U$10.P$8, U$10.P$9, U$11.P$1, U$11.P$10, U$11.P$11, U$11.P$12, U$11.P$2, U$11.P$3, U$11.P$4, U$11.P$5, U$11.P$6, U$11.P$7, U$11.P$8, U$11.P$9, U$12.P$1, U$12.P$10, U$12.P$11, U$12.P$12, U$12.P$2, U$12.P$3, U$12.P$4, U$12.P$5, U$12.P$6, U$12.P$7, U$12.P$8, U$12.P$9, U$13.P$1, U$13.P$10, U$13.P$11, U$13.P$12, U$13.P$2, U$13.P$3, U$13.P$4, U$13.P$5, U$13.P$6, U$13.P$7, U$13.P$8, U$13.P$9, U$3.P$1, U$3.P$10, U$3.P$11, U$3.P$12, U$3.P$2, U$3.P$3, U$3.P$4, U$3.P$5, U$3.P$6, U$3.P$7, U$3.P$8, U$3.P$9, U$9.P$1, U$9.P$10, U$9.P$11, U$9.P$12, U$9.P$2, U$9.P$3, U$9.P$4, U$9.P$5, U$9.P$6, U$9.P$7, U$9.P$8, U$9.P$9; no longer C5.1, C7.1, R4.1, U$2.P$2, X2.P$2, X3.P$2, X4.P$2, X5.P$2, X6.P$2
Routing:
- net VCC: track 107.0 -> 0.00 mm, vias 39 -> 38
- net AIN0: track 24.9 -> 0.00 mm
- net AIN1: track 21.0 -> 0.00 mm
- net AIN14: track 19.0 -> 0.00 mm
- net AIN2: track 17.0 -> 0.00 mm
- net AIN8: track 14.8 -> 0.00 mm
- net AIN13: track 14.5 -> 0.00 mm
- net AIN11: track 11.8 -> 0.00 mm
- net AIN12: track 11.6 -> 0.00 mm
- net AIN7: track 11.2 -> 0.00 mm
- net AIN3: track 9.13 -> 0.00 mm
- net AIN10: track 8.67 -> 0.00 mm
- net AIN6: track 8.18 -> 0.00 mm
- net AIN9: track 7.99 -> 0.00 mm
- net AIN4: track 5.16 -> 0.00 mm
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
Commit message: Connected connectors and thermistors to mux
Connected all the connectors and thermistors to each other, as well as
to the muxes and to the voltage divider resistors.
Parts:
- added R33, R34, R35, R36, R37, R38, R39, R4, R40, R41, R42, R43, R44, R45, R46, R47, R48, R49, R50, R51, R52, R53, R54, R55, R56, R57, R58, R59, R60, R61, R62, R63, R64, R65, R66, R67, R68, R69, R70, R71, R72, R73, R74, R75, R76, R77, R78, R79: 10K, adafruit:R0603
Connections:
- removed net AIN72: U$11.P$24
- removed net CS: IC1.39
- removed net DIN: IC1.42
- removed net DOUT: IC1.41
- removed net SCLK: IC1.40
- net AIN0: now also R55.1
- net AIN1: now also R54.1
- net AIN10: now also R13.1
- net AIN11: now also R14.1, U$12.P$24, U$4.P$19
- net AIN12: now also R15.1, U$13.P$13; no longer U$12.P$24, U$4.P$19
- net AIN13: now also R16.1, U$13.P$14; no longer U$13.P$13
- net AIN14: now also R17.1, U$13.P$15; no longer U$13.P$14
- net AIN15: now also R18.1, U$13.P$16; no longer U$13.P$15
- net AIN16: now also R19.1, U$13.P$17; no longer U$13.P$16
- net AIN17: now also R20.1, U$13.P$18; no longer U$13.P$17
- net AIN18: now also R4.1, U$13.P$19; no longer U$13.P$18
- net AIN19: now also R42.1, U$13.P$20; no longer U$13.P$19
- net AIN2: now also R53.1
- net AIN20: now also R43.1, U$13.P$21; no longer U$13.P$20
- net AIN21: now also R44.1, U$13.P$22; no longer U$13.P$21
- net AIN22: now also R45.1, U$13.P$23; no longer U$13.P$22
- net AIN23: now also R46.1, U$13.P$24; no longer U$13.P$23
- net AIN24: now also R49.1, U$3.P$13; no longer U$13.P$24
- net AIN25: now also R31.1, U$3.P$14; no longer U$3.P$13
- net AIN26: now also R32.1, U$3.P$15; no longer U$3.P$14
- net AIN27: now also R33.1, U$3.P$16; no longer U$3.P$15
- net AIN28: now also R34.1, U$3.P$17; no longer U$3.P$16
- net AIN29: now also R35.1, U$3.P$18; no longer U$3.P$17
- net AIN3: now also R52.1
- net AIN30: now also R36.1, U$3.P$19; no longer U$3.P$18
- net AIN31: now also R37.1, U$3.P$20; no longer U$3.P$19
- net AIN32: now also R38.1, U$3.P$21; no longer U$3.P$20
- net AIN33: now also R39.1, U$3.P$22; no longer U$3.P$21
- net AIN34: now also R40.1, U$3.P$23; no longer U$3.P$22
- net AIN35: now also R41.1, U$3.P$24; no longer U$3.P$23
- net AIN36: now also R61.1, U$9.P$13; no longer U$3.P$24
- net AIN37: now also R60.1, U$9.P$14; no longer U$9.P$13
- net AIN38: now also R59.1, U$9.P$15; no longer U$9.P$14
- net AIN39: now also R58.1, U$9.P$16; no longer U$9.P$15
- net AIN4: now also R51.1
- net AIN40: now also R57.1, U$9.P$17; no longer U$9.P$16
- net AIN41: now also R56.1, U$9.P$18; no longer U$9.P$17
- net AIN42: now also R21.1, U$9.P$19; no longer U$9.P$18
- net AIN43: now also R22.1, U$9.P$20; no longer U$9.P$19
- net AIN44: now also R23.1, U$9.P$21; no longer U$9.P$20
- net AIN45: now also R24.1, U$9.P$22; no longer U$9.P$21
- net AIN46: now also R25.1, U$9.P$23; no longer U$9.P$22
- net AIN47: now also R26.1, U$9.P$24; no longer U$9.P$23
- net AIN48: now also R29.1, U$10.P$13; no longer U$9.P$24
- net AIN49: now also R30.1, U$10.P$14; no longer U$10.P$13
- net AIN5: now also R50.1
- net AIN50: now also R27.1, U$10.P$15; no longer U$10.P$14
- net AIN51: now also R28.1, U$10.P$16; no longer U$10.P$15
- net AIN52: now also R47.1, U$10.P$17; no longer U$10.P$16
- net AIN53: now also R48.1, U$10.P$18; no longer U$10.P$17
- net AIN54: now also R62.1, U$10.P$19; no longer U$10.P$18
- net AIN55: now also R63.1, U$10.P$20; no longer U$10.P$19
- net AIN56: now also R64.1, U$10.P$21; no longer U$10.P$20
- net AIN57: now also R65.1, U$10.P$22; no longer U$10.P$21
- net AIN58: now also R66.1, U$10.P$23; no longer U$10.P$22
- net AIN59: now also R67.1, U$10.P$24; no longer U$10.P$23
- net AIN6: now also R5.1
- net AIN60: now also R68.1, U$11.P$13; no longer U$10.P$24
- net AIN61: now also R69.1, U$11.P$14; no longer U$11.P$13
- net AIN62: now also R70.1, U$11.P$15; no longer U$11.P$14
- net AIN63: now also R71.1, U$11.P$16; no longer U$11.P$15
- net AIN64: now also R72.1, U$11.P$17; no longer U$11.P$16
- net AIN65: now also R73.1, U$11.P$18; no longer U$11.P$17
- net AIN66: now also R74.1, U$11.P$19; no longer U$11.P$18
- net AIN67: now also R75.1, U$11.P$20; no longer U$11.P$19
- net AIN68: now also R76.1, U$11.P$21; no longer U$11.P$20
- net AIN69: now also R77.1, U$11.P$22; no longer U$11.P$21
- net AIN7: now also R10.1
- net AIN70: now also R78.1, U$11.P$23; no longer U$11.P$22
- net AIN71: now also R79.1, U$11.P$24; no longer U$11.P$23
- net AIN8: now also R11.1
- net AIN9: now also R12.1
- net GND: now also R33.2, R34.2, R35.2, R36.2, R37.2, R38.2, R39.2, R4.2, R40.2, R41.2, R42.2, R43.2, R44.2, R45.2, R46.2, R47.2, R48.2, R49.2, R50.2, R51.2, R52.2, R53.2, R54.2, R55.2, R56.2, R57.2, R58.2, R59.2, R60.2, R61.2, R62.2, R63.2, R64.2, R65.2, R66.2, R67.2, R68.2, R69.2, R70.2, R71.2, R72.2, R73.2, R74.2, R75.2, R76.2, R77.2, R78.2, R79.2
Routing:
- net CS: track 9.00 -> 0.00 mm
- net DIN: track 5.38 -> 0.00 mm
- net DOUT: track 5.26 -> 0.00 mm
- net SCLK: track 5.14 -> 0.00 mm
