File: EAGLE Models/BMS/BMS MiniCAN Boards/BMS MiniCAN Themistor Board Rev. 4.sch (EAGLE design)
At the start: 112 parts, among them IC1 AT90CAN128, IC2 MCP2551SO8, IC3 NUP2105L, U1 0ZCH0050FF2G

Commit message: Fixed silkscreens and crystal
Fixed the silkscreens and replaced crystal.
Parts:
- removed U$14: AX-16.000MBGE-T, BMS Lbr:AX-16.000MBGE-T
- added Y1: 16M, SparkFun-FreqCtrl:CRYSTALSMD
- renumbered SJ1 to JP1, U$1 to IC4, U$10 to X4, U$11 to X5, U$12 to X6, U$13 to X7, U$2 to X1, U$3 to X2, U$5 to IC5, U$6 to IC6, U$7 to IC7, U$8 to IC8, U$9 to X3, U1 to F1, VCC! to D4
Connections:
- net XTAL1: now also Y1.1; no longer U$14.P$1
- net XTAL2: now also Y1.2; no longer U$14.P$2

Commit message: Fixed resistor values
Fixed resistor values.
Parts:
- R10, R11, R12, R13, R14, R15, R16, R17, R18, R19, R20, R21, R22, R23, R24, R25, R26, R27, R28, R29, R30, R31, R32, R33, R34, R35, R36, R37, R38, R39, R4, R40, R41, R42, R43, R44, R45, R46, R47, R48, R49, R5, R50, R51, R52, R53, R54, R55, R56, R57, R58, R59, R60, R61, R62, R63, R64, R65, R66, R67, R68, R69, R70, R71, R72, R73, R74, R75, R76, R77, R78, R79: value (none) -> 10K
