File: EAGLE Models/BMS/BMS MiniCAN Boards/BMS MiniCAN Themistor Board Rev. 5.brd (EAGLE design)
At the start: 150.2 x 63.2 mm, 112 parts, among them IC1 AT90CAN128, IC2 MCP2551SO8, IC3 NUP2105L, IC4 LM117MPX-5.0, IC5 CD74HC4067, IC6 CD74HC4067, IC7 CD74HC4067, IC8 CD74HC4067, X1 10127720-241LF, X2 10127720-241LF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

Commit message: Changed various things
Changed hole sizes, rearranged protection circuit, changed mosi miso on
6 pin header, moved 6 pin header farther away from AT90, deleted
redundant protection diode, created better spacing for CAN protection
IC, added credits.
Parts:
- removed D2: DFLS1100, BMS Lbr:POWERDI-123
Connections:
- removed net 12VIN: C15.1, D2.P$1, IC4.P$3
- net 12V: now also C15.1, IC4.P$3; no longer D2.P$2
Routing:
- net 12V: track 48.4 -> 80.2 mm
- net 12VIN: track 28.3 -> 0.00 mm
