File: EAGLE Models/sbRIO Daughter Card/Daughter Card v6-shorter.brd (EAGLE design)
At the start: 153.7 x 102.9 mm, 96 parts, among them IC1 BTS716G, IC2 BTS716G, IC3 BTS716G

Commit message: moved components and connectors around and shortened the board
Parts:
- moved BSPD_U4 27.1 mm to (59.5, 27.0)
- moved AMS_U5 25.4 mm to (66.4, 27.0)
- moved IMD_U6 25.0 mm to (73.1, 27.0)
- moved F3 25.0 mm to (21.6, 16.5), turned to 180 degrees
- moved F1 21.8 mm to (59.8, 11.9)
- moved TSMS_CONN 21.2 mm to (48.7, 6.81)
- moved SAFETY_CONN 21.0 mm to (61.5, 6.88)
- moved LATCH_CONN 20.8 mm to (89.7, 6.88)
- moved AIO_PO_CONN 19.5 mm to (122.7, 81.8)
- moved F20 19.5 mm to (117.0, 76.7)
- moved R19 19.5 mm to (117.2, 50.6)
- moved R20 19.5 mm to (113.9, 45.4)
- moved R8 19.5 mm to (117.3, 82.1)
- moved TUB_CONN 19.5 mm to (122.7, 53.9)
- moved F15 19.5 mm to (117.0, 78.1)
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Routing:
- net AI1: track 242.7 -> 0.00 mm, vias 1 -> 0
- net E-STOP_OK: track 163.6 -> 2.64 mm, vias 2 -> 0
- net AI2: track 262.2 -> 101.7 mm, vias 2 -> 0
- net LATCH_OK: track 151.4 -> 2.32 mm, vias 2 -> 0
- net AMS_OK_IN: track 145.5 -> 2.54 mm, vias 1 -> 0
- net AO3: track 157.3 -> 35.7 mm, vias 2 -> 0
- net AI7: track 137.7 -> 16.5 mm
- net AO2: track 152.9 -> 33.3 mm, vias 2 -> 0
- net IMD_OK_IN: track 121.0 -> 2.39 mm, vias 2 -> 0
- net STEERING_POS: track 160.9 -> 43.3 mm
- net AO1: track 149.7 -> 32.1 mm, vias 2 -> 0
- net THROTTLE_IN_2: track 124.1 -> 7.31 mm
- net AO0: track 147.2 -> 31.5 mm, vias 2 -> 0
- net ACCUMULATOR_FANS: track 113.6 -> 0.00 mm
- net THROTTLE_IN_1: track 119.1 -> 8.12 mm
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- added copper zone on layer 1, net N$1
- removed copper zone on layer 1, net 12V
Other:
- board size 153.7 x 102.9 mm -> 137.8 x 102.9 mm

Commit message: started rerouting traces on the short board
Parts:
- moved C10 6.12 mm to (37.1, 28.5)
- moved C11 6.12 mm to (41.2, 28.4)
- moved C12 6.12 mm to (44.7, 28.4)
- moved C9 6.12 mm to (42.8, 25.4)
- moved U$3 6.12 mm to (41.9, 35.0)
- moved LATCH_U7 1.04 mm to (96.0, 66.9)
Routing:
- net DIO4: track 133.3 -> 0.00 mm, vias 3 -> 0
- net AI7: track 16.5 -> 124.3 mm
- net STEERING_POS: track 43.3 -> 148.5 mm
- net AO3: track 35.7 -> 140.1 mm, vias 0 -> 2
- net AO2: track 33.3 -> 136.7 mm, vias 0 -> 2
- net THROTTLE_IN_2: track 7.31 -> 110.3 mm
- net ACCUMULATOR_FANS: track 0.00 -> 102.0 mm
- net AO1: track 32.1 -> 133.6 mm, vias 0 -> 2
- net AO0: track 31.5 -> 131.3 mm, vias 0 -> 2
- net PO2: track 0.00 -> 97.5 mm
- net PO3: track 0.00 -> 96.7 mm
- net THROTTLE_IN_1: track 8.12 -> 103.5 mm
- net LATCH_SW_OUT: track 6.04 -> 43.3 mm
- net N$7: track 18.1 -> 50.4 mm
- net DIO_GND: track 218.9 -> 212.8 mm
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
Commit message: continued to run more traces and fixed drc errors
Parts:
- moved U$2 13.3 mm to (103.8, 75.9)
- moved R6 2.48 mm to (112.7, 84.8), turned to 180 degrees
- moved F16 2.24 mm to (104.2, 86.1), turned to 270 degrees
- moved U$1 2.15 mm to (87.5, 68.6), turned to 90 degrees
Routing:
- net AI2: track 101.7 -> 232.2 mm, vias 0 -> 2
- net 3.3V: track 169.6 -> 46.5 mm, vias 5 -> 3
- net IMD_OK_IN: track 2.39 -> 106.3 mm
- net AMS_OK_IN: track 2.54 -> 104.4 mm
- net 5V: track 121.5 -> 22.1 mm, vias 3 -> 1
- net PO4: track 1.59 -> 92.5 mm
- net CAN_GND: track 3.59 -> 92.6 mm
- net GLV+: track 38.3 -> 119.8 mm
- net CAN_H: track 0.00 -> 65.4 mm
- net CAN_L: track 0.00 -> 61.8 mm
- net DIO_GND: track 212.8 -> 163.9 mm, vias 4 -> 2
- net LAP_TIMER_IN: track 3.36 -> 42.3 mm, vias 0 -> 2
- net DC_DC_DISABLE: track 0.00 -> 32.0 mm, vias 0 -> 2
- net 5V_IO_1: track 0.00 -> 31.3 mm, vias 0 -> 2
- net LATCH_SW_IN: track 6.04 -> 34.1 mm
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- added copper zone on layer 1, net 12V
- removed copper zone on layer 1, net N$1
