File: EAGLE Models/sbRIO Daughter Card/Daughter Card v6.sch (EAGLE design)
At the start: 97 parts, among them IC1 BTS716G, IC10 MIC5225-3.3YM5-TR, IC11 MIC5225-3.3YM5-TR, IC12 MIC5225-3.3YM5-TR, IC2 BTS716G, IC3 BTS716G, IC8 MIC5225-3.3YM5-TR, IC9 MIC5225-3.3YM5-TR, K1 HE3621A1250_SPST, K2 HE3621A1250_SPST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

Commit message: connected the latch traces and the ams traces
Connections:
- net LATCH_OK: no longer IC8.3~16V_IN, R15.1
- net LATCH_SW_IN: now also IC8.3~16V_IN, R15.1
Changed lines of the file:
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@@
 <pinref part="AIO_PO_CONN" gate="-8" pin="KL"/>
-</segment>
-<segment>
-<pinref part="IC8" gate="G$1" pin="3~16V_IN"/>
-<wire x1="203.2" y1="-22.86" x2="223.52" y2="-22.86" width="0.1524" layer="91"/>
-<label x="223.52" y="-22.86" size="1.778" layer="95" xref="yes"/>
-<wire x1="203.2" y1="-22.86" x2="203.2" y2="-17.78" width="0.1524" layer="91"/>
-<junction x="203.2" y="-22.86"/>
-<pinref part="R15" gate="G$1" pin="1"/>
 </segment>
 </net>
@@
 </segment>
 <segment>
-<wire x1="215.9" y1="-27.94" x2="223.52" y2="-27.94" width="0.1524" layer="91"/>
-<label x="223.52" y="-27.94" size="1.778" layer="95" xref="yes"/>
+<label x="223.52" y="-22.86" size="1.778" layer="95" xref="yes"/>
+<pinref part="IC8" gate="G$1" pin="3~16V_IN"/>
+<wire x1="203.2" y1="-22.86" x2="203.2" y2="-17.78" width="0.1524" layer="91"/>
+<pinref part="R15" gate="G$1" pin="1"/>
+<wire x1="223.52" y1="-22.86" x2="203.2" y2="-22.86" width="0.1524" layer="91"/>
 </segment>
 </net>

Commit message: connected imd_ok+ to imd_ok_in
Connections:
- net IMD_OK+: now also IC10.3~16V_IN, R27.1
- net IMD_OK_IN: no longer IC10.3~16V_IN, R27.1
Changed lines of the file:
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@@
-</segment>
-</net>
-<net name="AMS_OK_IN" class="0">
-<segment>
-<pinref part="ACCUMULATOR_CONN" gate="G$1" pin="7"/>
-<wire x1="462.28" y1="-157.48" x2="429.26" y2="-157.48" width="0.1524" layer="91"/>
-<label x="429.26" y="-157.48" size="1.778" layer="95" rot="R180" xref="yes"/>
-</segment>
-<segment>
-<pinref part="IC9" gate="G$1" pin="3~16V_IN"/>
-<wire x1="203.2" y1="-10.16" x2="220.98" y2="-10.16" width="0.1524" layer="91"/>
-<wire x1="220.98" y1="-10.16" x2="220.98" y2="-5.08" width="0.1524" layer="91"/>
-<wire x1="220.98" y1="-5.08" x2="223.52" y2="-5.08" width="0.1524" layer="91"/>
-<label x="223.52" y="-5.08" size="1.778" layer="95" xref="yes"/>
-<pinref part="R1" gate="G$1" pin="1"/>
-<junction x="220.98" y="-10.16"/>
 </segment>
 </net>
@@
 <label x="447.04" y="-160.02" size="1.778" layer="95" rot="R180" xref="yes"/>
 </segment>
-<segment>
-<pinref part="IC10" gate="G$1" pin="3~16V_IN"/>
-<wire x1="203.2" y1="2.54" x2="223.52" y2="2.54" width="0.1524" layer="91"/>
-<label x="223.52" y="2.54" size="1.778" layer="95" xref="yes"/>
-<wire x1="203.2" y1="2.54" x2="203.2" y2="7.62" width="0.1524" layer="91"/>
-<junction x="203.2" y="2.54"/>
-<pinref part="R27" gate="G$1" pin="1"/>
-</segment>
 </net>
 <net name="DIO20" class="0">
@@
 <wire x1="728.98" y1="-27.94" x2="723.9" y2="-27.94" width="0.1524" layer="91"/>
 <label x="723.9" y="-27.94" size="1.778" layer="95" rot="R180" xref="yes"/>
+</segment>
+<segment>
+<pinref part="IC10" gate="G$1" pin="3~16V_IN"/>
+<wire x1="203.2" y1="2.54" x2="218.44" y2="2.54" width="0.1524" layer="91"/>
+<label x="223.52" y="2.54" size="1.778" layer="95" xref="yes"/>
+<wire x1="218.44" y1="2.54" x2="223.52" y2="2.54" width="0.1524" layer="91"/>
+<wire x1="203.2" y1="2.54" x2="203.2" y2="7.62" width="0.1524" layer="91"/>
+<junction x="203.2" y="2.54"/>
+<pinref part="R27" gate="G$1" pin="1"/>
+<wire x1="218.44" y1="2.54" x2="218.44" y2="7.62" width="0.1524" layer="91"/>
+<wire x1="218.44" y1="7.62" x2="226.06" y2="7.62" width="0.1524" layer="91"/>
+<label x="226.06" y="7.62" size="1.778" layer="95" xref="yes"/>
+<junction x="218.44" y="2.54"/>
 </segment>
 </net>
@@
 </segment>
 </net>
+<net name="AMS_OK_IN" class="0">
+<segment>
+<pinref part="ACCUMULATOR_CONN" gate="G$1" pin="7"/>
+<wire x1="462.28" y1="-157.48" x2="429.26" y2="-157.48" width="0.1524" layer="91"/>
+<label x="429.26" y="-157.48" size="1.778" layer="95" rot="R180" xref="yes"/>
+</segment>
+<segment>
+<pinref part="IC9" gate="G$1" pin="3~16V_IN"/>
+<wire x1="203.2" y1="-10.16" x2="220.98" y2="-10.16" width="0.1524" layer="91"/>
+<wire x1="220.98" y1="-10.16" x2="220.98" y2="-5.08" width="0.1524" layer="91"/>
+<wire x1="220.98" y1="-5.08" x2="223.52" y2="-5.08" width="0.1524" layer="91"/>
+<label x="223.52" y="-5.08" size="1.778" layer="95" xref="yes"/>
+<pinref part="R1" gate="G$1" pin="1"/>
+<junction x="220.98" y="-10.16"/>
+</segment>
+</net>

Commit message: routed imd_ok_in to imd_ok+
Connections:
- removed net IMD_OK_IN: ACCUMULATOR_CONN.8
- net AMS_OK-: now also ACCUMULATOR_CONN.7
- net AMS_OK_IN: no longer ACCUMULATOR_CONN.7
- net IMD_OK+: now also ACCUMULATOR_CONN.8
Changed lines of the file:
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@@
-</segment>
-</net>
-<net name="IMD_OK_IN" class="0">
-<segment>
-<wire x1="462.28" y1="-160.02" x2="447.04" y2="-160.02" width="0.1524" layer="91"/>
-<pinref part="ACCUMULATOR_CONN" gate="G$1" pin="8"/>
-<label x="447.04" y="-160.02" size="1.778" layer="95" rot="R180" xref="yes"/>
 </segment>
 </net>
@@
 <label x="236.22" y="-10.16" size="1.778" layer="95" xref="yes"/>
 </segment>
+<segment>
+<pinref part="ACCUMULATOR_CONN" gate="G$1" pin="7"/>
+<wire x1="462.28" y1="-157.48" x2="429.26" y2="-157.48" width="0.1524" layer="91"/>
+<label x="429.26" y="-157.48" size="1.778" layer="95" rot="R180" xref="yes"/>
+</segment>
 </net>
 <net name="IMD_OK+" class="0">
@@
 <label x="226.06" y="7.62" size="1.778" layer="95" xref="yes"/>
 <junction x="218.44" y="2.54"/>
+</segment>
+<segment>
+<wire x1="462.28" y1="-160.02" x2="447.04" y2="-160.02" width="0.1524" layer="91"/>
+<pinref part="ACCUMULATOR_CONN" gate="G$1" pin="8"/>
+<label x="447.04" y="-160.02" size="1.778" layer="95" rot="R180" xref="yes"/>
 </segment>
 </net>
@@
 <net name="AMS_OK_IN" class="0">
 <segment>
-<pinref part="ACCUMULATOR_CONN" gate="G$1" pin="7"/>
-<wire x1="462.28" y1="-157.48" x2="429.26" y2="-157.48" width="0.1524" layer="91"/>
-<label x="429.26" y="-157.48" size="1.778" layer="95" rot="R180" xref="yes"/>
-</segment>
-<segment>
 <pinref part="IC9" gate="G$1" pin="3~16V_IN"/>

Commit message: connected latch_ok to TSMS_out+ and e_stop_ok to TSMS_in+
Connections:
- net E-STOP_OK: no longer IC11.3~16V_IN, R28.1
- net LATCH_SW_IN: no longer IC8.3~16V_IN, R15.1
- net TSMS_IN+: now also IC11.3~16V_IN, R28.1
- net TSMS_OUT+: now also IC8.3~16V_IN, R15.1
Changed lines of the file:
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@@
 <net name="E-STOP_OK" class="0">
-<segment>
-<pinref part="IC11" gate="G$1" pin="3~16V_IN"/>
-<wire x1="203.2" y1="15.24" x2="223.52" y2="15.24" width="0.1524" layer="91"/>
-<label x="223.52" y="15.24" size="1.778" layer="95" xref="yes"/>
-<wire x1="203.2" y1="15.24" x2="203.2" y2="20.32" width="0.1524" layer="91"/>
-<junction x="203.2" y="15.24"/>
-<pinref part="R28" gate="G$1" pin="1"/>
-</segment>
 <segment>
 <wire x1="424.18" y1="-96.52" x2="462.28" y2="-96.52" width="0.1524" layer="91"/>
@@
 <label x="543.56" y="-127" size="1.778" layer="95" xref="yes"/>
 </segment>
-<segment>
-<label x="223.52" y="-22.86" size="1.778" layer="95" xref="yes"/>
-<pinref part="IC8" gate="G$1" pin="3~16V_IN"/>
-<wire x1="203.2" y1="-22.86" x2="203.2" y2="-17.78" width="0.1524" layer="91"/>
-<pinref part="R15" gate="G$1" pin="1"/>
-<wire x1="223.52" y1="-22.86" x2="203.2" y2="-22.86" width="0.1524" layer="91"/>
-</segment>
 </net>
 <net name="SHUTDOWN_OK+" class="0">
@@
 <label x="543.56" y="-96.52" size="1.778" layer="95" xref="yes"/>
 </segment>
+<segment>
+<label x="223.52" y="-22.86" size="1.778" layer="95" xref="yes"/>
+<pinref part="IC8" gate="G$1" pin="3~16V_IN"/>
+<wire x1="203.2" y1="-22.86" x2="203.2" y2="-17.78" width="0.1524" layer="91"/>
+<pinref part="R15" gate="G$1" pin="1"/>
+<wire x1="223.52" y1="-22.86" x2="218.44" y2="-22.86" width="0.1524" layer="91"/>
+<label x="223.52" y="-17.78" size="1.778" layer="95" xref="yes"/>
+<wire x1="218.44" y1="-22.86" x2="203.2" y2="-22.86" width="0.1524" layer="91"/>
+<wire x1="223.52" y1="-17.78" x2="218.44" y2="-17.78" width="0.1524" layer="91"/>
+<wire x1="218.44" y1="-17.78" x2="218.44" y2="-22.86" width="0.1524" layer="91"/>
+<junction x="218.44" y="-22.86"/>
+</segment>
 </net>
 <net name="TSMS_IN+" class="0">
@@
 <label x="541.02" y="-27.94" size="1.778" layer="95" xref="yes"/>
 </segment>
-</net>
+<segment>
+<pinref part="IC11" gate="G$1" pin="3~16V_IN"/>
+<wire x1="203.2" y1="15.24" x2="218.44" y2="15.24" width="0.1524" layer="91"/>
+<label x="223.52" y="15.24" size="1.778" layer="95" xref="yes"/>
+<wire x1="218.44" y1="15.24" x2="223.52" y2="15.24" width="0.1524" layer="91"/>
+<wire x1="203.2" y1="15.24" x2="203.2" y2="20.32" width="0.1524" layer="91"/>
+<junction x="203.2" y="15.24"/>
+<pinref part="R28" gate="G$1" pin="1"/>
+<label x="223.52" y="20.32" size="1.778" layer="95" xref="yes"/>
+<wire x1="223.52" y1="20.32" x2="218.44" y2="20.32" width="0.1524" layer="91"/>
+<wire x1="218.44" y1="20.32" x2="218.44" y2="15.24" width="0.1524" layer="91"/>
+<junction x="218.44" y="15.24"/>
+</segment>
+</net>

Commit message: fixed amd_ok-
Parts:
- removed R1: 10K, resistor:R-US_R0603
Connections:
- removed net AMS_OK_IN: IC9.3~16V_IN, R1.1
- net AMS_OK-: now also IC9.3~16V_IN; no longer R1.2
- net GLV+: no longer K5.C+
- net PO3: now also K5.C+
Changed lines of the file:
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@@
 <part name="R53" library="resistor" deviceset="R-US_" device="R0603" value="10K"/>
 <part name="GLV+_CONN" library="formula electric" deviceset="CONN_2" device=""/>
-<part name="R1" library="resistor" deviceset="R-US_" device="R0603" value="10K"/>
 </parts>
 <sheets>
@@
 <instance part="R53" gate="G$1" x="-86.36" y="-35.56"/>
 <instance part="GLV+_CONN" gate="G$1" x="530.86" y="-48.26"/>
-<instance part="R1" gate="G$1" x="226.06" y="-10.16"/>
 </instances>
 <busses>
@@
 <pinref part="AIO_PO_CONN" gate="-14" pin="KL"/>
 </segment>
+<segment>
+<pinref part="K5" gate="G$1" pin="C+"/>
+<wire x1="728.98" y1="-5.08" x2="723.9" y2="-5.08" width="0.1524" layer="91"/>
+<label x="723.9" y="-5.08" size="1.778" layer="95" rot="R180" xref="yes"/>
+</segment>
 </net>
 <net name="PO4" class="0">
@@
 </segment>
 <segment>
-<pinref part="R1" gate="G$1" pin="2"/>
-<wire x1="231.14" y1="-10.16" x2="236.22" y2="-10.16" width="0.1524" layer="91"/>
 <label x="236.22" y="-10.16" size="1.778" layer="95" xref="yes"/>
+<pinref part="IC9" gate="G$1" pin="3~16V_IN"/>
+<wire x1="203.2" y1="-10.16" x2="220.98" y2="-10.16" width="0.1524" layer="91"/>
+<wire x1="220.98" y1="-10.16" x2="220.98" y2="-5.08" width="0.1524" layer="91"/>
+<wire x1="220.98" y1="-5.08" x2="223.52" y2="-5.08" width="0.1524" layer="91"/>
+<label x="223.52" y="-5.08" size="1.778" layer="95" xref="yes"/>
+<wire x1="236.22" y1="-10.16" x2="220.98" y2="-10.16" width="0.1524" layer="91"/>
 </segment>
 <segment>
@@
 <wire x1="650.24" y1="20.32" x2="650.24" y2="25.4" width="0.1524" layer="91"/>
 <label x="650.24" y="25.4" size="1.778" layer="95" rot="R90" xref="yes"/>
-</segment>
-<segment>
-<pinref part="K5" gate="G$1" pin="C+"/>
-<wire x1="728.98" y1="-5.08" x2="723.9" y2="-5.08" width="0.1524" layer="91"/>
-<label x="723.9" y="-5.08" size="1.778" layer="95" rot="R180" xref="yes"/>
 </segment>
 <segment>
@@
 </segment>
 </net>
-<net name="AMS_OK_IN" class="0">
-<segment>
-<pinref part="IC9" gate="G$1" pin="3~16V_IN"/>
-<wire x1="203.2" y1="-10.16" x2="220.98" y2="-10.16" width="0.1524" layer="91"/>
-<wire x1="220.98" y1="-10.16" x2="220.98" y2="-5.08" width="0.1524" layer="91"/>
-<wire x1="220.98" y1="-5.08" x2="223.52" y2="-5.08" width="0.1524" layer="91"/>
-<label x="223.52" y="-5.08" size="1.778" layer="95" xref="yes"/>
-<pinref part="R1" gate="G$1" pin="1"/>
-<junction x="220.98" y="-10.16"/>
-</segment>
-</net>

Commit message: made the changes that thomas suggested
adjusted many of the high side driver- connector signals and moved the
dimentions to silkscreen
Parts:
- R39, R40, R41, R42, R43, R44, R45, R46, R47, R48, R49, R50, R51, R52, R53: value 10K -> 100k
Connections:
- net AMS_OUT renamed BRAKELIGHT
- removed net BSPD_OUT: IC3G$1.OUT4, TUB_CONN-4.KL
- removed net LATCH_OK: AIO_PO_CONN-8.KL
- removed net PO2: AIO_PO_CONN-15.KL, IC1G$1.OUT2
- removed net PO4: AIO_PO_CONN-13.KL, IC1G$1.OUT4
- removed net SHUTDOWN_1: IC2G$1.OUT2
- new net COOLANT_PUMP: AIO_PO_CONN-13.KL, IC1G$1.OUT2
- new net FAN_PWM_OUT: AIO_PO_CONN-16.KL, IC3G$1.OUT4, TUB_CONN-4.KL
- net ACCUMULATOR_FANS: now also AIO_PO_CONN-15.KL; no longer AIO_PO_CONN-16.KL
- net AMS_OK-: no longer ACCUMULATOR_CONN.7
- net PRECHARGE_DONE+: now also AIO_PO_CONN-8.KL, IC1G$1.OUT4
- net SBRIO_OK+_2: now also IC2G$1.OUT2
Changed lines of the file:
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@@
 <part name="R37" library="resistor" deviceset="R-US_" device="R0603" value="10K"/>
 <part name="R38" library="resistor" deviceset="R-US_" device="R0603" value="10K"/>
-<part name="R39" library="resistor" deviceset="R-US_" device="R0603" value="10K"/>
-<part name="R40" library="resistor" deviceset="R-US_" device="R0603" value="10K"/>
-<part name="R41" library="resistor" deviceset="R-US_" device="R0603" value="10K"/>
-<part name="R42" library="resistor" deviceset="R-US_" device="R0603" value="10K"/>
-<part name="R43" library="resistor" deviceset="R-US_" device="R0603" value="10K"/>
-<part name="R44" library="resistor" deviceset="R-US_" device="R0603" value="10K"/>
-<part name="R45" library="resistor" deviceset="R-US_" device="R0603" value="10K"/>
-<part name="R46" library="resistor" deviceset="R-US_" device="R0603" value="10K"/>
-<part name="R47" library="resistor" deviceset="R-US_" device="R0603" value="10K"/>
-<part name="R48" library="resistor" deviceset="R-US_" device="R0603" value="10K"/>
-<part name="R49" library="resistor" deviceset="R-US_" device="R0603" value="10K"/>
-<part name="R50" library="resistor" deviceset="R-US_" device="R0603" value="10K"/>
-<part name="R51" library="resistor" deviceset="R-US_" device="R0603" value="10K"/>
-<part name="R52" library="resistor" deviceset="R-US_" device="R0603" value="10K"/>
-<part name="R53" library="resistor" deviceset="R-US_" device="R0603" value="10K"/>
+<part name="R39" library="resistor" deviceset="R-US_" device="R0603" value="100k"/>
+<part name="R40" library="resistor" deviceset="R-US_" device="R0603" value="100k"/>
+<part name="R41" library="resistor" deviceset="R-US_" device="R0603" value="100k"/>
+<part name="R42" library="resistor" deviceset="R-US_" device="R0603" value="100k"/>
+<part name="R43" library="resistor" deviceset="R-US_" device="R0603" value="100k"/>
+<part name="R44" library="resistor" deviceset="R-US_" device="R0603" value="100k"/>
+<part name="R45" library="resistor" deviceset="R-US_" device="R0603" value="100k"/>
+<part name="R46" library="resistor" deviceset="R-US_" device="R0603" value="100k"/>
+<part name="R47" library="resistor" deviceset="R-US_" device="R0603" value="100k"/>
+<part name="R48" library="resistor" deviceset="R-US_" device="R0603" value="100k"/>
+<part name="R49" library="resistor" deviceset="R-US_" device="R0603" value="100k"/>
+<part name="R50" library="resistor" deviceset="R-US_" device="R0603" value="100k"/>
+<part name="R51" library="resistor" deviceset="R-US_" device="R0603" value="100k"/>
+<part name="R52" library="resistor" deviceset="R-US_" device="R0603" value="100k"/>
+<part name="R53" library="resistor" deviceset="R-US_" device="R0603" value="100k"/>
 <part name="GLV+_CONN" library="formula electric" deviceset="CONN_2" device=""/>
 </parts>
@@
 </segment>
 </net>
-<net name="AMS_OUT" class="0">
-<segment>
-<wire x1="350.52" y1="-137.16" x2="350.52" y2="-142.24" width="0.1524" layer="91"/>
-<label x="350.52" y="-142.24" size="1.778" layer="95" rot="R270" xref="yes"/>
-<pinref part="IC3" gate="G$1" pin="OUT2"/>
-</segment>
-<segment>
-<wire x1="462.28" y1="-27.94" x2="449.58" y2="-27.94" width="0.1524" layer="91"/>
-<label x="449.58" y="-27.94" size="1.778" layer="95" rot="R180" xref="yes"/>
-<pinref part="TUB_CONN" gate="-6" pin="KL"/>
-</segment>
-</net>
 <net name="IMD_OUT" class="0">
 <segment>
@@
 <label x="421.64" y="-30.48" size="1.778" layer="95" rot="R180" xref="yes"/>
 <pinref part="TUB_CONN" gate="-5" pin="KL"/>
-</segment>
-</net>
-<net name="BSPD_OUT" class="0">
-<segment>
-<wire x1="337.82" y1="-137.16" x2="337.82" y2="-142.24" width="0.1524" layer="91"/>
-<label x="337.82" y="-142.24" size="1.778" layer="95" rot="R270" xref="yes"/>
-<pinref part="IC3" gate="G$1" pin="OUT4"/>
-</segment>
-<segment>
-<wire x1="462.28" y1="-33.02" x2="449.58" y2="-33.02" width="0.1524" layer="91"/>
-<label x="449.58" y="-33.02" size="1.778" layer="95" rot="R180" xref="yes"/>
-<pinref part="TUB_CONN" gate="-4" pin="KL"/>
 </segment>
 </net>
@@
 </segment>
 <segment>
-<label x="421.64" y="-66.04" size="1.778" layer="95" rot="R180" xref="yes"/>
-<pinref part="AIO_PO_CONN" gate="-16" pin="KL"/>
-<wire x1="462.28" y1="-66.04" x2="421.64" y2="-66.04" width="0.1524" layer="91"/>
-</segment>
-</net>
-<net name="PO2" class="0">
-<segment>
-<label x="279.4" y="-142.24" size="1.778" layer="95" rot="R270" xref="yes"/>
-<wire x1="279.4" y1="-137.16" x2="279.4" y2="-142.24" width="0.1524" layer="91"/>
-<pinref part="IC1" gate="G$1" pin="OUT2"/>
-</segment>
-<segment>
-<wire x1="462.28" y1="-68.58" x2="436.88" y2="-68.58" width="0.1524" layer="91"/>
-<label x="436.88" y="-68.58" size="1.778" layer="95" rot="R180" xref="yes"/>
 <pinref part="AIO_PO_CONN" gate="-15" pin="KL"/>
+<wire x1="462.28" y1="-68.58" x2="421.64" y2="-68.58" width="0.1524" layer="91"/>
+<label x="421.64" y="-68.58" size="1.778" layer="95" rot="R180" xref="yes"/>
 </segment>
 </net>
@@
 </segment>
 <segment>
-<wire x1="462.28" y1="-71.12" x2="421.64" y2="-71.12" width="0.1524" layer="91"/>
-<label x="421.64" y="-71.12" size="1.778" layer="95" rot="R180" xref="yes"/>
+<label x="429.26" y="-71.12" size="1.778" layer="95" rot="R180" xref="yes"/>
 <pinref part="AIO_PO_CONN" gate="-14" pin="KL"/>
+<wire x1="429.26" y1="-71.12" x2="462.28" y2="-71.12" width="0.1524" layer="91"/>
 </segment>
 <segment>
@@
 </segment>
 </net>
-<net name="PO4" class="0">
-<segment>
-<wire x1="266.7" y1="-137.16" x2="266.7" y2="-142.24" width="0.1524" layer="91"/>
-<label x="266.7" y="-142.24" size="1.778" layer="95" rot="R270" xref="yes"/>
-<pinref part="IC1" gate="G$1" pin="OUT4"/>
-</segment>
-<segment>
-<wire x1="462.28" y1="-73.66" x2="436.88" y2="-73.66" width="0.1524" layer="91"/>
-<label x="436.88" y="-73.66" size="1.778" layer="95" rot="R180" xref="yes"/>
-<pinref part="AIO_PO_CONN" gate="-13" pin="KL"/>
-</segment>
-</net>
 <net name="N$3" class="0">
 <segment>
@@
 <label x="302.26" y="-142.24" size="1.778" layer="95" rot="R270" xref="yes"/>
 <pinref part="IC2" gate="G$1" pin="OUT4"/>
-</segment>
-</net>
-<net name="SHUTDOWN_1" class="0">
-<segment>
-<wire x1="314.96" y1="-137.16" x2="314.96" y2="-142.24" width="0.1524" layer="91"/>
-<label x="314.96" y="-142.24" size="1.778" layer="95" rot="R270" xref="yes"/>
-<pinref part="IC2" gate="G$1" pin="OUT2"/>
 </segment>
 </net>
@@
 <label x="424.18" y="-96.52" size="1.778" layer="95" rot="R180" xref="yes"/>
 <pinref part="AIO_PO_CONN" gate="-4" pin="KL"/>
-</segment>
-</net>
-<net name="LATCH_OK" class="0">
-<segment>
-<wire x1="462.28" y1="-86.36" x2="424.18" y2="-86.36" width="0.1524" layer="91"/>
-<label x="424.18" y="-86.36" size="1.778" layer="95" rot="R180" xref="yes"/>
-<pinref part="AIO_PO_CONN" gate="-8" pin="KL"/>
 </segment>
 </net>
@@
 <wire x1="236.22" y1="-10.16" x2="220.98" y2="-10.16" width="0.1524" layer="91"/>
 </segment>
-<segment>
-<pinref part="ACCUMULATOR_CONN" gate="G$1" pin="7"/>
-<wire x1="462.28" y1="-157.48" x2="429.26" y2="-157.48" width="0.1524" layer="91"/>
-<label x="429.26" y="-157.48" size="1.778" layer="95" rot="R180" xref="yes"/>
-</segment>
 </net>
 <net name="IMD_OK+" class="0">
@@
 <label x="378.46" y="43.18" size="1.778" layer="95" rot="R180" xref="yes"/>
 </segment>
+<segment>
+<wire x1="462.28" y1="-86.36" x2="424.18" y2="-86.36" width="0.1524" layer="91"/>
+<label x="424.18" y="-86.36" size="1.778" layer="95" rot="R180" xref="yes"/>
+<pinref part="AIO_PO_CONN" gate="-8" pin="KL"/>
+</segment>
+<segment>
+<wire x1="266.7" y1="-137.16" x2="266.7" y2="-142.24" width="0.1524" layer="91"/>
+<label x="266.7" y="-142.24" size="1.778" layer="95" rot="R270" xref="yes"/>
+<pinref part="IC1" gate="G$1" pin="OUT4"/>
+</segment>
 </net>
 <net name="GLV+" class="0">
@@
 <pinref part="F14" gate="G$1" pin="1"/>
 <label x="624.84" y="0" size="1.778" layer="95" rot="R180" xref="yes"/>
+</segment>
+<segment>
+<wire x1="314.96" y1="-137.16" x2="314.96" y2="-142.24" width="0.1524" layer="91"/>
+<label x="314.96" y="-142.24" size="1.778" layer="95" rot="R270" xref="yes"/>
+<pinref part="IC2" gate="G$1" pin="OUT2"/>
 </segment>
 </net>
@@
 </segment>
 </net>
+<net name="BRAKELIGHT" class="0">
+<segment>
+<wire x1="350.52" y1="-137.16" x2="350.52" y2="-142.24" width="0.1524" layer="91"/>
+<label x="350.52" y="-142.24" size="1.778" layer="95" rot="R270" xref="yes"/>
+<pinref part="IC3" gate="G$1" pin="OUT2"/>
+</segment>
+<segment>
+<wire x1="462.28" y1="-27.94" x2="449.58" y2="-27.94" width="0.1524" layer="91"/>
+<label x="449.58" y="-27.94" size="1.778" layer="95" rot="R180" xref="yes"/>
+<pinref part="TUB_CONN" gate="-6" pin="KL"/>
+</segment>
+</net>
+<net name="FAN_PWM_OUT" class="0">
+<segment>
+<label x="444.5" y="-66.04" size="1.778" layer="95" rot="R180" xref="yes"/>
+<pinref part="AIO_PO_CONN" gate="-16" pin="KL"/>
+<wire x1="462.28" y1="-66.04" x2="444.5" y2="-66.04" width="0.1524" layer="91"/>
+</segment>
+<segment>
+<wire x1="462.28" y1="-33.02" x2="449.58" y2="-33.02" width="0.1524" layer="91"/>
+<label x="449.58" y="-33.02" size="1.778" layer="95" rot="R180" xref="yes"/>
+<pinref part="TUB_CONN" gate="-4" pin="KL"/>
+</segment>
+<segment>
+<wire x1="337.82" y1="-137.16" x2="337.82" y2="-142.24" width="0.1524" layer="91"/>
+<label x="337.82" y="-142.24" size="1.778" layer="95" rot="R270" xref="yes"/>
+<pinref part="IC3" gate="G$1" pin="OUT4"/>
+</segment>
+</net>
+<net name="COOLANT_PUMP" class="0">
+<segment>
+<label x="279.4" y="-142.24" size="1.778" layer="95" rot="R270" xref="yes"/>
+<wire x1="279.4" y1="-137.16" x2="279.4" y2="-142.24" width="0.1524" layer="91"/>
+<pinref part="IC1" gate="G$1" pin="OUT2"/>
+</segment>
+<segment>
+<pinref part="AIO_PO_CONN" gate="-13" pin="KL"/>
+<wire x1="462.28" y1="-73.66" x2="421.64" y2="-73.66" width="0.1524" layer="91"/>
+<label x="421.64" y="-73.66" size="1.778" layer="95" rot="R180" xref="yes"/>
+</segment>
+</net>
