File: EAGLE Models/sbRIO Daughter Card/Daughter Card v6.sch (EAGLE design)
At the start: 96 parts, among them IC1 BTS716G, IC10 MIC5225-3.3YM5-TR, IC11 MIC5225-3.3YM5-TR, IC12 MIC5225-3.3YM5-TR, IC2 BTS716G, IC3 BTS716G, IC8 MIC5225-3.3YM5-TR, IC9 MIC5225-3.3YM5-TR, K1 HE3621A1250_SPST, K2 HE3621A1250_SPST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

Commit message: changed the spare trace from the high side driver to right angle conn to PO2
Connections:
- net IMD_OUT renamed PO2
- net FAN_PWM_OUT: no longer TUB_CONN-4.KL
Changed lines of the file:
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@@
-</segment>
-</net>
-<net name="IMD_OUT" class="0">
-<segment>
-<wire x1="342.9" y1="-137.16" x2="342.9" y2="-142.24" width="0.1524" layer="91"/>
-<label x="342.9" y="-142.24" size="1.778" layer="95" rot="R270" xref="yes"/>
-<pinref part="IC3" gate="G$1" pin="OUT3"/>
-</segment>
-<segment>
-<wire x1="462.28" y1="-30.48" x2="421.64" y2="-30.48" width="0.1524" layer="91"/>
-<label x="421.64" y="-30.48" size="1.778" layer="95" rot="R180" xref="yes"/>
-<pinref part="TUB_CONN" gate="-5" pin="KL"/>
 </segment>
 </net>
@@
 <label x="236.22" y="-10.16" size="1.778" layer="95" xref="yes"/>
 <pinref part="IC9" gate="G$1" pin="3~16V_IN"/>
-<wire x1="203.2" y1="-10.16" x2="220.98" y2="-10.16" width="0.1524" layer="91"/>
-<wire x1="220.98" y1="-10.16" x2="220.98" y2="-5.08" width="0.1524" layer="91"/>
-<wire x1="220.98" y1="-5.08" x2="223.52" y2="-5.08" width="0.1524" layer="91"/>
-<label x="223.52" y="-5.08" size="1.778" layer="95" xref="yes"/>
-<wire x1="236.22" y1="-10.16" x2="220.98" y2="-10.16" width="0.1524" layer="91"/>
+<wire x1="203.2" y1="-10.16" x2="236.22" y2="-10.16" width="0.1524" layer="91"/>
 </segment>
 </net>
@@
 <segment>
 <pinref part="IC10" gate="G$1" pin="3~16V_IN"/>
-<wire x1="203.2" y1="2.54" x2="218.44" y2="2.54" width="0.1524" layer="91"/>
+<wire x1="203.2" y1="2.54" x2="223.52" y2="2.54" width="0.1524" layer="91"/>
 <label x="223.52" y="2.54" size="1.778" layer="95" xref="yes"/>
-<wire x1="218.44" y1="2.54" x2="223.52" y2="2.54" width="0.1524" layer="91"/>
 <wire x1="203.2" y1="2.54" x2="203.2" y2="7.62" width="0.1524" layer="91"/>
 <junction x="203.2" y="2.54"/>
 <pinref part="R27" gate="G$1" pin="1"/>
-<wire x1="218.44" y1="2.54" x2="218.44" y2="7.62" width="0.1524" layer="91"/>
-<wire x1="218.44" y1="7.62" x2="226.06" y2="7.62" width="0.1524" layer="91"/>
-<label x="226.06" y="7.62" size="1.778" layer="95" xref="yes"/>
-<junction x="218.44" y="2.54"/>
 </segment>
 <segment>
@@
 <wire x1="203.2" y1="-22.86" x2="203.2" y2="-17.78" width="0.1524" layer="91"/>
 <pinref part="R15" gate="G$1" pin="1"/>
-<wire x1="223.52" y1="-22.86" x2="218.44" y2="-22.86" width="0.1524" layer="91"/>
-<label x="223.52" y="-17.78" size="1.778" layer="95" xref="yes"/>
-<wire x1="218.44" y1="-22.86" x2="203.2" y2="-22.86" width="0.1524" layer="91"/>
-<wire x1="223.52" y1="-17.78" x2="218.44" y2="-17.78" width="0.1524" layer="91"/>
-<wire x1="218.44" y1="-17.78" x2="218.44" y2="-22.86" width="0.1524" layer="91"/>
-<junction x="218.44" y="-22.86"/>
+<wire x1="223.52" y1="-22.86" x2="203.2" y2="-22.86" width="0.1524" layer="91"/>
 </segment>
 </net>
@@
 <segment>
 <pinref part="IC11" gate="G$1" pin="3~16V_IN"/>
-<wire x1="203.2" y1="15.24" x2="218.44" y2="15.24" width="0.1524" layer="91"/>
+<wire x1="203.2" y1="15.24" x2="223.52" y2="15.24" width="0.1524" layer="91"/>
 <label x="223.52" y="15.24" size="1.778" layer="95" xref="yes"/>
-<wire x1="218.44" y1="15.24" x2="223.52" y2="15.24" width="0.1524" layer="91"/>
 <wire x1="203.2" y1="15.24" x2="203.2" y2="20.32" width="0.1524" layer="91"/>
 <junction x="203.2" y="15.24"/>
 <pinref part="R28" gate="G$1" pin="1"/>
-<label x="223.52" y="20.32" size="1.778" layer="95" xref="yes"/>
-<wire x1="223.52" y1="20.32" x2="218.44" y2="20.32" width="0.1524" layer="91"/>
-<wire x1="218.44" y1="20.32" x2="218.44" y2="15.24" width="0.1524" layer="91"/>
-<junction x="218.44" y="15.24"/>
 </segment>
 </net>
@@
 </segment>
 <segment>
-<wire x1="462.28" y1="-33.02" x2="449.58" y2="-33.02" width="0.1524" layer="91"/>
-<label x="449.58" y="-33.02" size="1.778" layer="95" rot="R180" xref="yes"/>
-<pinref part="TUB_CONN" gate="-4" pin="KL"/>
-</segment>
-<segment>
 <wire x1="337.82" y1="-137.16" x2="337.82" y2="-142.24" width="0.1524" layer="91"/>
 <label x="337.82" y="-142.24" size="1.778" layer="95" rot="R270" xref="yes"/>
@@
 </segment>
 </net>
+<net name="PO2" class="0">
+<segment>
+<wire x1="462.28" y1="-30.48" x2="421.64" y2="-30.48" width="0.1524" layer="91"/>
+<label x="421.64" y="-30.48" size="1.778" layer="95" rot="R180" xref="yes"/>
+<pinref part="TUB_CONN" gate="-5" pin="KL"/>
+</segment>
+<segment>
+<wire x1="342.9" y1="-137.16" x2="342.9" y2="-142.24" width="0.1524" layer="91"/>
+<label x="342.9" y="-142.24" size="1.778" layer="95" rot="R270" xref="yes"/>
+<pinref part="IC3" gate="G$1" pin="OUT3"/>
+</segment>
+</net>

Commit message: added tps7a4533 voltage regulator to library
did not yet add to board
Parts:
- C11: value 10uF -> 0.1uF
- C12: value 22uF -> 0.22uF
Changed lines of the file:
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@@
 <part name="C10" library="SparkFun-Passives" deviceset="CAP" device="0603-CAP" value="10uF"/>
 <part name="C9" library="SparkFun-Passives" deviceset="CAP" device="0603-CAP" value="22uF"/>
-<part name="C11" library="SparkFun-Passives" deviceset="CAP" device="0603-CAP" value="10uF"/>
-<part name="C12" library="SparkFun-Passives" deviceset="CAP" device="0603-CAP" value="22uF"/>
+<part name="C11" library="SparkFun-Passives" deviceset="CAP" device="0603-CAP" value="0.1uF"/>
+<part name="C12" library="SparkFun-Passives" deviceset="CAP" device="0603-CAP" value="0.22uF"/>
 <part name="ACCEL" library="SparkFun-Sensors" deviceset="ADXL345" device=""/>
 <part name="C7" library="SparkFun-Passives" deviceset="CAP" device="0603-CAP" value=".1uF"/>
