File: EAGLE Models/sbRIO Daughter Card/Daughter Card v5.brd (EAGLE design)
At the start: 101.6 x 81.3 mm, 83 parts, among them IC1 BTS716G, IC2 BTS716G, IC3 BTS716G

Commit message: renamed trace to have better name
Connections:
- net 5V_FUSED renamed N$20
- net SHUTDOWN_1_FUSED renamed N$15
- net SHUTDOWN_2_FUSED renamed N$12

Commit message: changed some net names
changed the N$__ nets to be descriptive
Connections:
- net N$12 renamed SHUTDOWN_2_FUSED
- net N$15 renamed SHUTDOWN_1_FUSED
- net N$20 renamed 5V_FUSED
