File: EAGLE Models/sbRIO Daughter Card/Daughter Card v5.sch (EAGLE design)
At the start: 83 parts, among them IC1 BTS716G, IC2 BTS716G, IC3 BTS716G

Commit message: changed some net names
changed the N$__ nets to be descriptive
Connections:
- net N$12 renamed SHUTDOWN_2_FUSED
- net N$15 renamed SHUTDOWN_1_FUSED
- net N$20 renamed 5V_FUSED
Changed lines of the file:
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@@
 <?xml version="1.0" encoding="utf-8"?>
 <!DOCTYPE eagle SYSTEM "eagle.dtd">
-<eagle version="7.2.0">
+<eagle version="7.7.0">
 <drawing>
 <settings>
@@
 </segment>
 </net>
-<net name="N$20" class="0">
+<net name="5V_FUSED" class="0">
 <segment>
 <pinref part="F16" gate="G$1" pin="2"/>
@@
 </segment>
 </net>
-<net name="N$12" class="0">
+<net name="SHUTDOWN_2_FUSED" class="0">
 <segment>
 <pinref part="F2" gate="G$1" pin="2"/>
@@
 </segment>
 </net>
-<net name="N$15" class="0">
+<net name="SHUTDOWN_1_FUSED" class="0">
 <segment>
 <pinref part="F14" gate="G$1" pin="2"/>

Commit message: renamed trace to have better name
Connections:
- net 5V_FUSED renamed N$20
- net SHUTDOWN_1_FUSED renamed N$15
- net SHUTDOWN_2_FUSED renamed N$12
Changed lines of the file:
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@@
 <?xml version="1.0" encoding="utf-8"?>
 <!DOCTYPE eagle SYSTEM "eagle.dtd">
-<eagle version="7.7.0">
+<eagle version="7.2.0">
 <drawing>
 <settings>
@@
 </segment>
 </net>
-<net name="5V_FUSED" class="0">
+<net name="N$20" class="0">
 <segment>
 <pinref part="F16" gate="G$1" pin="2"/>
@@
 </segment>
 </net>
-<net name="SHUTDOWN_2_FUSED" class="0">
+<net name="N$12" class="0">
 <segment>
 <pinref part="F2" gate="G$1" pin="2"/>
@@
 </segment>
 </net>
-<net name="SHUTDOWN_1_FUSED" class="0">
+<net name="N$15" class="0">
 <segment>
 <pinref part="F14" gate="G$1" pin="2"/>
