File: EAGLE Models/sbRIO Daughter Card/Daughter Card v7.sch (EAGLE design)
At the start: 88 parts, among them IC1 BTS716G, IC2 BTS716G, IC3 BTS716G

Commit message: Began Seriously reworking Daughter card and tracing nets to new connectors
Parts:
- removed TUB_CONN: 2516-5, con-3m:2516-5
- added F4: 0.5A PTC, resistor:R-EU_R0603
- added F5, F7, F8, F9: 10mA PTC, resistor:R-EU_R0402
- added U$7: SULLINS_1MM_6P_HEADER, formula electric:SULLINS_1MM_6P_HEADER
Connections:
- new net BRAKELIGHT: U$6.A17
- new net COOLANT_PUMP: AIO_PO_CONN-13.KL
- new net FAN_PWM_OUT: AIO_PO_CONN-16.KL
- new net N$11: U$6.A22
- new net N$12: F4.2
- new net N$15: U$6.B3
- new net N$16: U$6.A4
- new net N$17: U$6.A5
- new net N$18: U$6.A6
- new net N$19: U$6.A7
- new net N$21: U$6.A8
- new net N$22: U$6.A9
- new net N$23: U$6.B4
- new net N$24: U$6.B5
- new net N$25: U$6.B6
- new net N$26: U$6.B7
- new net N$28: U$6.A19
- new net N$30: U$6.A20
- new net N$31: U$6.B9
- new net N$32: U$6.B10
- new net N$33: U$6.A23
- new net N$34: U$6.A24
- new net N$35: U$6.A25
- new net N$36: U$6.A26
- new net N$37: U$6.A27
- new net N$38: U$6.A28
- new net N$39: U$6.A29
- new net N$40: U$6.A30
- new net N$42: U$6.A31
- new net N$43: U$6.A32
- new net N$44: U$6.A33
- new net N$45: U$6.A34
- new net N$67: U$6.B11
- new net N$68: U$6.B12
- new net N$69: U$6.B13
- new net N$70: F5.2
- new net N$71: F7.2
- new net N$72: F8.2
- new net N$73: F9.2
- net 5V: now also F4.1
- net 5V_IO_1: no longer TUB_CONN-3.KL
- net ACCUMULATOR_FANS: now also AIO_PO_CONN-15.KL; no longer AIO_PO_CONN-16.KL
- net AI7: now also U$6.A11; no longer TUB_CONN-15.KL
- net AMS_OUT: no longer TUB_CONN-6.KL
- net AO0: now also F5.1
- net AO1: now also F7.1
- net AO2: now also F8.1
- net AO3: now also F9.1
- net BRAKE_PRESS_IN_1: now also U$6.A15; no longer TUB_CONN-11.KL
- net BRAKE_PRESS_IN_2: now also U$6.A14; no longer TUB_CONN-12.KL
- net BSPD_OUT: no longer TUB_CONN-4.KL
- net BUZZER_OUT: now also U$6.A16; no longer TUB_CONN-7.KL
- net CAN_GND: now also U$6.A3; no longer TUB_CONN-10.KL
- net CAN_H: now also U$6.A1, U$6.B1; no longer TUB_CONN-9.KL
- net CAN_L: now also U$6.A2, U$6.B2; no longer TUB_CONN-8.KL
- net DC_DC_DISABLE: now also U$6.B8; no longer TUB_CONN-1.KL
- net IMD_OUT: no longer TUB_CONN-5.KL
- net LAP_TIMER_IN: now also U$6.A21; no longer TUB_CONN-2.KL
- net LATCH_OK: no longer AIO_PO_CONN-8.KL
- net PO2: now also U$6.A18; no longer AIO_PO_CONN-15.KL
- net PO4: no longer AIO_PO_CONN-13.KL
- net PRECHARGE_DONE+: now also AIO_PO_CONN-8.KL
- net STEERING_POS: now also U$6.A10; no longer TUB_CONN-16.KL
- net THROTTLE_IN_1: now also U$6.A13; no longer TUB_CONN-13.KL
- net THROTTLE_IN_2: now also U$6.A12; no longer TUB_CONN-14.KL
Other:
- note added: "connections to PDM"

Commit message: Worked more on remapping connectors on daughter card
Parts:
- removed AIO_PO_CONN: 2516-5, con-3m:2516-5
- removed AMS_U5, BSPD_U4, IMD_U6, INTERLOCKS_U3, SBRIO_U1, SBRIO_U2: HE3621A1250_SPST, formula electric:HE3621A1250_SPST
- removed F14, F2: 250mA, resistor:R-EU_R0603
- removed F15, F20, F21, F22: 10mA PTC, resistor:R-EU_R0402
- removed F16: 0.5A PTC, resistor:R-EU_R0603
- removed F3: FUSEX20MM, SparkFun-Passives:FUSEX20MM
- removed LATCH_CONN, SAFETY_CONN: CONN_5, formula electric:CONN_5
- removed LATCH_U7: JW2SN-DC12V, formula electric:JW2SN-DC12V
- removed TSMS_CONN: CONN_2, formula electric:CONN_2
- removed U$1, U$2: DIODE_MMBD4448, formula electric:DIODE_MMBD4448
- removed U$8: RELAY, formula electric:RELAY
- added D7, D8: DIODE_MMBD4448, formula electric:DIODE_MMBD4448
- added F10, F11: 250mA, resistor:R-EU_R0603
- added F12: FUSEX20MM, SparkFun-Passives:FUSEX20MM
- added GLV+_CONN, TSMS_CONN1: CONN_2, formula electric:CONN_2
- added K1, K2, K3, K4, K5, K6: HE3621A1250_SPST, formula electric:HE3621A1250_SPST
- added LATCH_CONN1, SAFETY_CONN1: CONN_5, formula electric:CONN_5
- added LATCH_U1: JW2SN-DC12V, formula electric:JW2SN-DC12V
- added U$9: RELAY, formula electric:RELAY
Connections:
- removed net COOLANT_PUMP: AIO_PO_CONN-13.KL
- removed net FAN_PWM_OUT: AIO_PO_CONN-16.KL
- removed net N$13: AMS_U5.SW_2, IMD_U6.SW_1
- removed net N$14: F3.1, U$8.A
- removed net N$16: U$6.A4
- removed net N$17: U$6.A5
- removed net N$18: U$6.A6
- removed net N$19: U$6.A7
- removed net N$2: SBRIO_U1.SW_2, SBRIO_U2.SW_1
- removed net N$20: AIO_PO_CONN-2.KL, F16.2
- removed net N$21: U$6.A8
- removed net N$22: U$6.A9
- removed net N$29: AIO_PO_CONN-3.KL
- removed net N$44: U$6.A33
- removed net N$7: INTERLOCKS_U3.SW_1, SBRIO_U2.SW_2
- removed net N$8: AMS_U5.SW_1, BSPD_U4.SW_2
- removed net SBRIO_OK+_1_RELAY_IN: F2.2, SBRIO_U1.C+
- removed net SBRIO_OK_2_RELAY: F14.2, SBRIO_U2.C+
- new net K4: K4.SW_2, K5.SW_1
- new net N$46: U$6.B14
- new net N$47: U$6.B15
- new net N$48: U$6.B16
- new net N$49: U$6.B17
- new net N$50: U$6.B18
- new net N$51: U$6.B19
- new net N$53: U$6.B22
- new net N$55: U$6.B23
- new net N$59: U$6.B24
- new net N$65: U$6.B26
- new net SBRIO_OK+_1_RELAY_IN1: F10.2, K3.C+
- new net SBRIO_OK_2_RELAY1: F11.2, K2.C+
- net 5V: no longer F16.1
- net ACCUMULATOR_FANS: no longer AIO_PO_CONN-15.KL
- net AI10: now also U$6.A6; no longer AIO_PO_CONN-7.KL
- net AI8: now also U$6.A8; no longer AIO_PO_CONN-5.KL
- net AI9: now also U$6.A7; no longer AIO_PO_CONN-6.KL
- net AMS_OK-: now also K5.C-, SAFETY_CONN1.2; no longer AMS_U5.C+, SAFETY_CONN.2
- net AO0: no longer F15.1
- net AO1: no longer F20.1
- net AO2: no longer F21.1
- net AO3: no longer F22.1
- net BSPD_OK+: now also K4.C+, SAFETY_CONN1.5; no longer BSPD_U4.C+, SAFETY_CONN.1
- net CAN_GND: no longer U$6.A3
- net CAN_H: now also U$6.A33, U$6.B20; no longer U$6.A1, U$6.B1
- net CAN_L: now also U$6.A34, U$6.B21; no longer U$6.A2, U$6.B2
- net E-STOP_OK: no longer AIO_PO_CONN-4.KL
- net GLV+: now also F12.2, GLV+_CONN.2, K3.SW_1, K4.SW_1; no longer AMS_U5.C-, BSPD_U4.SW_1, F3.2, SBRIO_U1.SW_1
- net GND: now also D7.A, D8.A, K1.C-, K2.C-, K3.C-, K4.C-, K6.C-, LATCH_CONN1.4, LATCH_U1.C_1, U$9.V1; no longer BSPD_U4.C-, IMD_U6.C-, INTERLOCKS_U3.C-, LATCH_CONN.4, LATCH_U7.C_1, SBRIO_U1.C-, SBRIO_U2.C-, U$1.A, U$2.A, U$8.V1
- net IMD_OK+: now also K6.C+, SAFETY_CONN1.3; no longer IMD_U6.C+, SAFETY_CONN.3
- net INTER_OK+: now also K1.C+, SAFETY_CONN1.4; no longer INTERLOCKS_U3.C+, SAFETY_CONN.4
- net LATCH_LED+: now also LATCH_CONN1.3, LATCH_U1.NC_2; no longer LATCH_CONN.3, LATCH_U7.NC_2
- net LATCH_SW_IN: now also D7.C, LATCH_CONN1.1, LATCH_U1.C_2, LATCH_U1.NO_2; no longer LATCH_CONN.1, LATCH_U7.C_2, LATCH_U7.NO_2, U$1.C
- net LATCH_SW_OUT: now also K6.SW_2, LATCH_CONN1.2, LATCH_U1.IN_2; no longer IMD_U6.SW_2, LATCH_CONN.2, LATCH_U7.IN_2
- net N$10: now also F12.1, U$9.A; no longer AIO_PO_CONN-12.KL, F22.2
- net N$12: now also U$6.A9
- net N$3: now also K2.SW_1, K3.SW_2; no longer AIO_PO_CONN-9.KL, F15.2
- net N$45: now also U$6.B2; no longer U$6.A34
- net N$6: now also K1.SW_1, K2.SW_2; no longer AIO_PO_CONN-10.KL, F20.2
- net N$70: now also U$6.A4
- net N$71: now also U$6.A3
- net N$72: now also U$6.A2
- net N$73: now also U$6.A1
- net N$9: now also K5.SW_2, K6.SW_1; no longer AIO_PO_CONN-11.KL, F21.2
- net PO3: now also K5.C+; no longer AIO_PO_CONN-14.KL
- net PRECHARGE_DONE+: now also TSMS_CONN1.2, U$6.A5; no longer AIO_PO_CONN-8.KL, TSMS_CONN.2
- net SBRIO_OK+_1: now also F10.1; no longer F2.1
- net SBRIO_OK+_2: now also F11.1; no longer F14.1
- net SHUTDOWN_OK+: now also K1.SW_2, LATCH_U1.NO_1; no longer INTERLOCKS_U3.SW_2, LATCH_U7.NO_1
- net TSMS_IN+: now also TSMS_CONN1.1; no longer TSMS_CONN.1
- net TSMS_OUT+: now also SAFETY_CONN1.1, U$9.C; no longer SAFETY_CONN.5, U$8.C
- net TSMS_OUT_CTRL+: now also D8.C, LATCH_U1.IN_1, U$9.V2; no longer LATCH_U7.IN_1, U$2.C, U$8.V2
Other:
- moved on the sheet: F4, F5, F7, F8, F9

Commit message: Almost done remapping signals, and created board to start laying out
Parts:
- removed ACCUMULATOR_CONN: RJ45-6L21-S, con-tycoelectronics:RJ45-6L21-S
- removed SBRIO_CAN: SBRIO_W500, formula electric:SBRIO_W500
- added U$1: SBRIO_BMS_CONN, formula electric:SBRIO_BMS_CONN
Connections:
- removed net AI1: ACCUMULATOR_CONN.2, R24.2, SBRIO_ANALOG.AI1
- removed net AI2: ACCUMULATOR_CONN.3, BSPD_CONN.4, R25.2, SBRIO_ANALOG.AI2
- removed net CAN_GND: ACCUMULATOR_CONN.1, ACCUMULATOR_CONN.S@1, ACCUMULATOR_CONN.S@2, ACCUMULATOR_CONN.S@3, ACCUMULATOR_CONN.S@4, SBRIO_CAN.V-_(GND)
- removed net N$36: U$6.A26
- removed net N$37: U$6.A27
- removed net SHIELD: ACCUMULATOR_CONN.6, SBRIO_CAN.SHIELD
- new net HIGH_CURRENT_IN: R24.2, SBRIO_ANALOG.AI1, U$6.A26
- new net LOW_CURRENT_IN: BSPD_CONN.4, R25.2, SBRIO_ANALOG.AI2, U$6.A27
- new net N$13: U$1.P$7
- new net N$16: U$1.P$1
- new net N$17: U$1.P$2
- new net N$18: U$1.P$3
- new net N$19: U$1.P$4
- new net N$20: U$1.P$5
- new net N$8: U$1.P$8
- net AMS_OK_IN: no longer ACCUMULATOR_CONN.7
- net CAN_H: now also U$1.P$10; no longer ACCUMULATOR_CONN.5, SBRIO_CAN.CAN_H
- net CAN_L: now also U$1.P$9; no longer ACCUMULATOR_CONN.4, SBRIO_CAN.CAN_L
- net IMD_OK_IN: no longer ACCUMULATOR_CONN.8
Other:
- note added: "BSPD CONN"
- note removed: "sbRIO CAN ribbon connector"
- moved on the sheet: SAFETY_CONN1, U$7
