File: EAGLE Models/Battery Characterizer/Battery Characterizer.sch (EAGLE design)
At the start: 92 parts, among them IC5 FT232RL, T1 IPB80P03P4L-04, T2 IPB80P03P4L-04, T3 IPB80P03P4L-04, T5 IRF40B207, T7 NTF6P02, U1 ATMEGA328P, U2 INA199A1DCKR, U3 INA199A1DCKR, U4 MIC4416YM4-TR, U5 KA378R05TU, U6 ADR5045AKSZ-REEL7, U7 TLV2556IPW, X1 MINI-USB-UX60-MB-5S8

Commit message: Finalized Schematic
Removed 3rd battery conn due to layout difficulties and cost increase
Parts:
- removed D5, D6: RA_13V1, Sanken:RA_13V1
- removed U7: TLV2556IPW, Texas Instruments_By_element14_Batch_1:TLV2556IPW
- added BATT_4, LOAD_2: CONN_2, formula electric:CONN_2
- added C26, C28: 10uF, rcl:C-USC0603
- added C29, C30, C31, C32, C33, C34, C35, C36, C38: 0.1uF, rcl:C-USC0603
- added C37: 4.7uF, rcl:C-USC0603
- added F5: PTC_FUSE, LittleFuse:PTC_FUSE
- added PC2: MCP73826, microchip:MCP73826
- added R20, R21, R32, R33, R34, R35: 100k, rcl:R-US_M0805
- added R22, R24, R25, R8: 10k, resistor:R-US_R0603
- added R23: 0R005, vishay:WSL3637
- added R26: 0R047, resistor:R-US_M1206
- added R27: 18k, resistor:R-US_R0603
- added R28: 2.2k, resistor:R-US_R0603
- added T4: IPB80P03P4L-04, infineon:IPB80P03P4L-04
- added T6: IRF40B207, infineon:IRF40B207
- added T8: NTF6P02, ON Semiconductor_By_element14_Batch_1:NTF6P02
- added U$6: IRLML6401TRPBF, International_Rectifier_By_element14_Batch_1:IRLML6401TRPBF
- added U$7: ADC128S022CIMTX/NOPB, texas:ADC128S022CIMTX/NOPB
- added U10: MIC4416YM4-TR, Microchip_By_element14_Batch_1:MIC4416YM4-TR
- added U8, U9: INA199A1DCKR, Texas Instruments_By_element14_Batch_1:INA199A1DCKR
- D4: value RA_13V1 -> 12TQ045; device Sanken:RA_13V1 -> SMC_Diode:12TQ045
- R7: value 100k -> 10k; device rcl:R-US_M0805 -> resistor:R-US_R0603; PN RL1220T-R039 -> RC0603FR-0710KL
Connections:
- removed net BATT_CONN_3_1: BATT_3.1, D6.C, F4.2
- removed net BATT_EN_3_1: R7.2, T3.G, U1.ADC6
- removed net BATT_EN_3_2: U1.PD7(AIN1)
- removed net CHARGE_1: C4.1, T7.D, U$3.S, U$4.S, U$5.S
- removed net FUSE_OUT_3_2: F4.1, T3.S
- removed net N$1: D4.A, U$3.D
- removed net N$2: D5.A, U$4.D
- removed net N$3: D6.A, U$5.D
- removed net N$8: U1.PD2(INT0)
- removed net N$9: U1.PD3(INT1)
- removed net PMOS_OUT_3_1: D3.A, T3.D
- new net BATT+_2: D3.C, D4.C, R23.1, R8.1
- new net BATT_CONN_1_2: BATT_3.1, F5.2
- new net BATT_CONN_2_2: BATT_4.1, F4.2
- new net CHARGE_1_1: R21.2, U$3.G, U1.PD2(INT0)
- new net CHARGE_1_2: R35.2, U$5.G, U1.PB0(ICP)
- new net CHARGE_2_1: R20.1, U$4.G, U1.PD3(INT1)
- new net CHARGE_2_2: R34.1, U$6.G, U1.PB1(OC1A)
- new net CHARGE_MAIN_1: C4.1, PC1.V_BAT, T7.D, U$3.S, U$4.S
- new net CHARGE_MAIN_2: C28.1, PC2.V_BAT, T8.D, U$5.S, U$6.S
- new net CHARGE_REF_2: R27.2, R28.1, U9.REF
- new net DISC_GATE_2: T6.G, U10.G
- new net DISC_INV_2: C32.1, R22.2, U8.IN-
- new net DISC_NON_INV_2: C31.1, R8.2, U8.IN+
- new net FUSE_OUT_1_2: F5.1, T3.S
- new net FUSE_OUT_2_2: F4.1, T4.S
- new net GATE_2: PC2.V_DRV, T8.G
- new net INV_2: C35.1, R24.2, U9.IN-
- new net LOAD+_2: LOAD_2.2, R22.1, R23.2
- new net NMOS_IN_2: LOAD_2.1, T6.D
- new net NON_INV_2: C36.1, R25.2, U9.IN+
- new net PMOS_OUT_1_2: D4.A, T3.D, U$5.D
- new net PMOS_OUT_2_2: D3.A, T4.D, U$6.D
- new net SHDN_2: PC2.SHDN, R7.1
- new net V_SNS_2: PC2.V_SNS, R24.1, R26.2, T8.S
- net 12V: now also C37.1, C38.1, U10.VS
- net AVCC: now also U$7.VA; no longer U7.REF+
- net BATT+_1: no longer D3.C, PC1.V_BAT
- net BATT_CONN_1_1: now also U$7.IN0; no longer D4.C, U7.AIN0
- net BATT_CONN_2_1: now also U$7.IN1; no longer D5.C, U7.AIN1
- net BATT_CONN_3: now also U$7.IN4; no longer U7.AIN4
- net BATT_CONN_4: now also U$7.IN5; no longer U7.AIN5
- net BATT_EN_1_2: now also R32.2, T3.G, U1.PD4(XCK/T0); no longer U1.PD5(T1)
- net BATT_EN_2_2: now also R33.2, T4.G, U1.PD5(T1); no longer U1.PD6(AIN0)
- net CHARGE_EN_1: now also U1.ADC6
- net CHARGE_EN_2: now also R7.2, U1.PD6(AIN0); no longer U1.ADC7, U1.PB0(ICP)
- net CHARGE_SENSE_1: now also U$7.IN2; no longer U7.AIN3
- net CHARGE_SENSE_2: now also C34.1, U$7.IN6, U9.OUT; no longer U7.AIN2
- net CS0: now also U$7.CS; no longer U7.~CS
- net DISC_EN_1: now also U1.ADC7; no longer U1.PD4(XCK/T0)
- net DISC_EN_2: now also U1.PD7(AIN1), U10.CTL; no longer U1.PB1(OC1A)
- net GND: now also BATT_4.2, C26.2, C28.2, C29.2, C30.2, C31.2, C32.2, C33.2, C34.2, C35.2, C36.2, C37.2, C38.2, PC2.GND, R28.2, T6.S, U$7.AGND, U$7.DGND, U10.GND, U8.GND, U8.REF, U9.GND; no longer U7.GND, U7.REF-
- net I_SENSE_1: now also U$7.IN3; no longer U7.AIN6
- net I_SENSE_2: now also C30.1, U$7.IN7, U8.OUT; no longer U7.AIN7
- net MISO: now also U$7.VD; no longer U7.DATA_OUT
- net MOSI: now also U$7.DIN; no longer U7.DATA_IN
- net PMOS_OUT_1_1: now also U$3.D
- net PMOS_OUT_2_1: now also U$4.D
- net SCK: now also U$7.SCLK; no longer U7.I/O_CLOCK
- net VCC: now also C26.1, C29.1, C33.1, PC2.V_IN, R20.2, R21.1, R25.1, R26.1, R27.1, R32.1, R33.1, R34.2, R35.1, U$7.DOUT, U8.V+, U9.V+; no longer R7.1, U7.VCC
Other:
- moved on the sheet: BATT_1, BATT_2, BATT_3, C14, C15, C23, C24, D1, D2, D3, D4, F1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

Commit message: Board Layout Improvements. Changed Charging Mosfet from obsolete one
Parts:
- removed C31, C32, C35, C36: 0.1uF, rcl:C-USC0603
- removed U$1: AX-16.000MBGE-T, BMS Lbr:AX-16.000MBGE-T
- added Q1: 56P2859, SparkFun-FreqCtrl:CRYSTALSMD
- C1, C18, C2, C37: device rcl:C-USC0603 -> rcl:C-USC0805
- C12: value 0.1uF -> 10uF
- C24: device resistor:C-USC0805 -> rcl:C-USC0805
- T1, T2, T3, T4: value IPB80P03P4L-04 -> IPP80P03P4L04AKSA1; device infineon:IPB80P03P4L-04 -> infineon:IPP80P03P4L04AKSA1
- T7, T8: value NTF6P02 -> STD28P3LLH6AG; device ON Semiconductor_By_element14_Batch_1:NTF6P02 -> st-microelectronics:STD28P3LLH6AG
- renumbered U$3 to T9, U$4 to T10, U$5 to T11, U$6 to T12
Connections:
- net BATT_EN_1_2: now also U1.PD7(AIN1); no longer U1.PD4(XCK/T0)
- net BATT_EN_2_2: now also U1.PD4(XCK/T0); no longer U1.PD5(T1)
- net CHARGE_1_1: now also U1.PD5(T1); no longer U1.PD2(INT0)
- net CHARGE_2_1: now also U1.PB1(OC1A); no longer U1.PD3(INT1)
- net CHARGE_2_2: now also U1.PD3(INT1); no longer U1.PB1(OC1A)
- net DISC_EN_2: now also U1.PD2(INT0); no longer U1.PD7(AIN1)
- net DISC_INV_1: now also C11.2; no longer C8.1
- net DISC_INV_2: now also C8.2; no longer C32.1
- net DISC_NON_INV_1: now also C11.1; no longer C7.1
- net DISC_NON_INV_2: now also C8.1; no longer C31.1
- net GND: no longer C11.2, C12.2, C31.2, C32.2, C35.2, C36.2, C7.2, C8.2
- net INV_1: now also C12.2; no longer C11.1
- net INV_2: now also C7.2; no longer C35.1
- net NON_INV_2: now also C7.1; no longer C36.1
- net XTAL1: now also Q1.2; no longer U$1.P$2
- net XTAL2: now also Q1.1; no longer U$1.P$1
Other:
- moved on the sheet: C11, C12, C7, C8

Commit message: Added correct mosfet, put vias through pads for thermals, changed pinout for better routing
Connections:
- net BATT_EN_1_1: now also U1.PB0(ICP); no longer U1.PC0(ADC0)
- net BATT_EN_1_2: now also U1.PD3(INT1); no longer U1.PD7(AIN1)
- net BATT_EN_2_1: now also U1.PD6(AIN0); no longer U1.PC1(ADC1)
- net BATT_EN_2_2: now also U1.PC1(ADC1); no longer U1.PD4(XCK/T0)
- net CHARGE_1_1: now also U1.PB1(OC1A); no longer U1.PD5(T1)
- net CHARGE_1_2: now also U1.PD2(INT0); no longer U1.PB0(ICP)
- net CHARGE_2_1: now also U1.PD5(T1); no longer U1.PB1(OC1A)
- net CHARGE_2_2: now also U1.PC0(ADC0); no longer U1.PD3(INT1)
- net CHARGE_EN_2: now also U1.PD4(XCK/T0); no longer U1.PD6(AIN0)
- net DISC_EN_1: now also U1.PD7(AIN1); no longer U1.ADC7
- net DISC_EN_2: now also U1.ADC7; no longer U1.PD2(INT0)
Changed lines of the file:
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@@
 </segment>
 <segment>
-<pinref part="U1" gate="G$1" pin="ADC7"/>
-<wire x1="17.78" y1="22.86" x2="22.86" y2="22.86" width="0.1524" layer="91"/>
-<label x="22.86" y="22.86" size="1.27" layer="95" font="vector" xref="yes"/>
+<pinref part="U1" gate="G$1" pin="PD7(AIN1)"/>
+<wire x1="17.78" y1="0" x2="22.86" y2="0" width="0.1524" layer="91"/>
+<label x="22.86" y="0" size="1.27" layer="95" font="vector" xref="yes"/>
 </segment>
 </net>
@@
 </segment>
 <segment>
-<pinref part="U1" gate="G$1" pin="PC0(ADC0)"/>
-<wire x1="17.78" y1="40.64" x2="22.86" y2="40.64" width="0.1524" layer="91"/>
-<label x="22.86" y="40.64" size="1.27" layer="95" font="vector" xref="yes"/>
+<pinref part="U1" gate="G$1" pin="PB0(ICP)"/>
+<wire x1="17.78" y1="-5.08" x2="22.86" y2="-5.08" width="0.1524" layer="91"/>
+<label x="22.86" y="-5.08" size="1.27" layer="95" font="vector" xref="yes"/>
 </segment>
 </net>
@@
 </segment>
 <segment>
-<pinref part="U1" gate="G$1" pin="PC1(ADC1)"/>
-<wire x1="17.78" y1="38.1" x2="22.86" y2="38.1" width="0.1524" layer="91"/>
-<label x="22.86" y="38.1" size="1.27" layer="95" font="vector" xref="yes"/>
+<pinref part="U1" gate="G$1" pin="PD6(AIN0)"/>
+<wire x1="17.78" y1="2.54" x2="22.86" y2="2.54" width="0.1524" layer="91"/>
+<label x="22.86" y="2.54" size="1.27" layer="95" font="vector" xref="yes"/>
 </segment>
 </net>
@@
 </segment>
 <segment>
-<pinref part="U1" gate="G$1" pin="PD7(AIN1)"/>
-<wire x1="17.78" y1="0" x2="22.86" y2="0" width="0.1524" layer="91"/>
-<label x="22.86" y="0" size="1.27" layer="95" font="vector" xref="yes"/>
+<pinref part="U1" gate="G$1" pin="PD3(INT1)"/>
+<wire x1="17.78" y1="10.16" x2="22.86" y2="10.16" width="0.1524" layer="91"/>
+<label x="22.86" y="10.16" size="1.27" layer="95" font="vector" xref="yes"/>
 </segment>
 </net>
@@
 </segment>
 <segment>
+<pinref part="U1" gate="G$1" pin="PC1(ADC1)"/>
+<wire x1="17.78" y1="38.1" x2="22.86" y2="38.1" width="0.1524" layer="91"/>
+<label x="22.86" y="38.1" size="1.27" layer="95" font="vector" xref="yes"/>
+</segment>
+</net>
+<net name="CHARGE_EN_2" class="0">
+<segment>
+<pinref part="R7" gate="G$1" pin="2"/>
+<wire x1="-302.26" y1="111.76" x2="-299.72" y2="111.76" width="0.1524" layer="91"/>
+<label x="-299.72" y="111.76" size="1.27" layer="95" font="vector" xref="yes"/>
+</segment>
+<segment>
 <pinref part="U1" gate="G$1" pin="PD4(XCK/T0)"/>
 <wire x1="17.78" y1="7.62" x2="22.86" y2="7.62" width="0.1524" layer="91"/>
@@
 </segment>
 </net>
-<net name="CHARGE_EN_2" class="0">
-<segment>
-<pinref part="U1" gate="G$1" pin="PD6(AIN0)"/>
-<wire x1="17.78" y1="2.54" x2="22.86" y2="2.54" width="0.1524" layer="91"/>
-<label x="22.86" y="2.54" size="1.27" layer="95" font="vector" xref="yes"/>
-</segment>
-<segment>
-<pinref part="R7" gate="G$1" pin="2"/>
-<wire x1="-302.26" y1="111.76" x2="-299.72" y2="111.76" width="0.1524" layer="91"/>
-<label x="-299.72" y="111.76" size="1.27" layer="95" font="vector" xref="yes"/>
-</segment>
-</net>
 <net name="DISC_EN_2" class="0">
 <segment>
@@
 </segment>
 <segment>
-<pinref part="U1" gate="G$1" pin="PD2(INT0)"/>
-<wire x1="17.78" y1="12.7" x2="22.86" y2="12.7" width="0.1524" layer="91"/>
-<label x="22.86" y="12.7" size="1.27" layer="95" font="vector" xref="yes"/>
+<pinref part="U1" gate="G$1" pin="ADC7"/>
+<wire x1="17.78" y1="22.86" x2="22.86" y2="22.86" width="0.1524" layer="91"/>
+<label x="22.86" y="22.86" size="1.27" layer="95" font="vector" xref="yes"/>
 </segment>
 </net>
@@
 </segment>
 <segment>
-<pinref part="U1" gate="G$1" pin="PB1(OC1A)"/>
-<wire x1="17.78" y1="-7.62" x2="22.86" y2="-7.62" width="0.1524" layer="91"/>
-<label x="22.86" y="-7.62" size="1.27" layer="95" font="vector" xref="yes"/>
+<pinref part="U1" gate="G$1" pin="PD5(T1)"/>
+<wire x1="17.78" y1="5.08" x2="22.86" y2="5.08" width="0.1524" layer="91"/>
+<label x="22.86" y="5.08" size="1.27" layer="95" font="vector" xref="yes"/>
 </segment>
 </net>
@@
 </segment>
 <segment>
-<pinref part="U1" gate="G$1" pin="PD5(T1)"/>
-<wire x1="17.78" y1="5.08" x2="22.86" y2="5.08" width="0.1524" layer="91"/>
-<label x="22.86" y="5.08" size="1.27" layer="95" font="vector" xref="yes"/>
+<pinref part="U1" gate="G$1" pin="PB1(OC1A)"/>
+<wire x1="17.78" y1="-7.62" x2="22.86" y2="-7.62" width="0.1524" layer="91"/>
+<label x="22.86" y="-7.62" size="1.27" layer="95" font="vector" xref="yes"/>
 </segment>
 </net>
 <net name="CHARGE_1_2" class="0">
-<segment>
-<pinref part="U1" gate="G$1" pin="PB0(ICP)"/>
-<wire x1="17.78" y1="-5.08" x2="22.86" y2="-5.08" width="0.1524" layer="91"/>
-<label x="22.86" y="-5.08" size="1.27" layer="95" font="vector" xref="yes"/>
-</segment>
 <segment>
 <pinref part="R35" gate="G$1" pin="2"/>
@@
 <label x="-373.38" y="-12.7" size="1.27" layer="95" font="vector" rot="R180" xref="yes"/>
 </segment>
+<segment>
+<pinref part="U1" gate="G$1" pin="PD2(INT0)"/>
+<wire x1="17.78" y1="12.7" x2="22.86" y2="12.7" width="0.1524" layer="91"/>
+<label x="22.86" y="12.7" size="1.27" layer="95" font="vector" xref="yes"/>
+</segment>
 </net>
 <net name="CHARGE_2_2" class="0">
@@
 </segment>
 <segment>
-<pinref part="U1" gate="G$1" pin="PD3(INT1)"/>
-<wire x1="17.78" y1="10.16" x2="22.86" y2="10.16" width="0.1524" layer="91"/>
-<label x="22.86" y="10.16" size="1.27" layer="95" font="vector" xref="yes"/>
-</segment>
-</net>
+<pinref part="U1" gate="G$1" pin="PC0(ADC0)"/>
+<wire x1="17.78" y1="40.64" x2="22.86" y2="40.64" width="0.1524" layer="91"/>
+<label x="22.86" y="40.64" size="1.27" layer="95" font="vector" xref="yes"/>
+</segment>
+</net>

Commit message: Layed Out Power Traces for Discharge and Charge Section. Needs Main Power In and Control Signals Routed
Connections:
- removed net BATT_CONN_3: U$7.IN4
- removed net BATT_CONN_4: U$7.IN5
- net BATT_CONN_1_1: now also U$7.IN4; no longer U$7.IN0
- net BATT_CONN_1_2: now also U$7.IN0
- net BATT_CONN_2_1: now also U$7.IN6; no longer U$7.IN1
- net BATT_CONN_2_2: now also U$7.IN5
- net BATT_EN_1_1: now also U1.ADC6; no longer U1.PB0(ICP)
- net CHARGE_EN_1: now also U1.PB0(ICP); no longer U1.ADC6
- net CHARGE_SENSE_2: now also U$7.IN1; no longer U$7.IN6
Changed lines of the file:
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@@
 </segment>
 <segment>
-<pinref part="U1" gate="G$1" pin="ADC6"/>
-<wire x1="17.78" y1="25.4" x2="22.86" y2="25.4" width="0.1524" layer="91"/>
-<label x="22.86" y="25.4" size="1.27" layer="95" font="vector" xref="yes"/>
+<pinref part="U1" gate="G$1" pin="PB0(ICP)"/>
+<wire x1="17.78" y1="-5.08" x2="22.86" y2="-5.08" width="0.1524" layer="91"/>
+<label x="22.86" y="-5.08" size="1.27" layer="95" font="vector" xref="yes"/>
 </segment>
 </net>
@@
 <net name="CHARGE_SENSE_2" class="0">
 <segment>
-<wire x1="-17.78" y1="60.96" x2="-15.24" y2="60.96" width="0.1524" layer="91"/>
-<label x="-15.24" y="60.96" size="1.27" layer="95" font="vector" xref="yes"/>
-<pinref part="U$7" gate="G$1" pin="IN6"/>
-</segment>
-<segment>
 <pinref part="U9" gate="A" pin="OUT"/>
 <wire x1="-347.98" y1="22.86" x2="-350.52" y2="22.86" width="0.1524" layer="91"/>
@@
 <wire x1="-350.52" y1="20.32" x2="-350.52" y2="22.86" width="0.1524" layer="91"/>
 <junction x="-350.52" y="22.86"/>
+</segment>
+<segment>
+<label x="-40.64" y="66.04" size="1.27" layer="95" font="vector" rot="R180" xref="yes"/>
+<wire x1="-40.64" y1="66.04" x2="-38.1" y2="66.04" width="0.1524" layer="91"/>
+<pinref part="U$7" gate="G$1" pin="IN1"/>
 </segment>
 </net>
@@
 <net name="BATT_CONN_1_1" class="0">
 <segment>
-<label x="-40.64" y="68.58" size="1.27" layer="95" font="vector" rot="R180" xref="yes"/>
-<wire x1="-40.64" y1="68.58" x2="-38.1" y2="68.58" width="0.1524" layer="91"/>
-<pinref part="U$7" gate="G$1" pin="IN0"/>
-</segment>
-<segment>
 <pinref part="F2" gate="G$1" pin="2"/>
 <pinref part="BATT_1" gate="G$1" pin="1"/>
@@
 <label x="-220.98" y="-22.86" size="1.27" layer="95" font="vector" xref="yes"/>
 </segment>
+<segment>
+<label x="-40.64" y="58.42" size="1.27" layer="95" font="vector" rot="R180" xref="yes"/>
+<wire x1="-40.64" y1="58.42" x2="-38.1" y2="58.42" width="0.1524" layer="91"/>
+<pinref part="U$7" gate="G$1" pin="IN4"/>
+</segment>
 </net>
 <net name="BATT_CONN_2_1" class="0">
-<segment>
-<label x="-40.64" y="66.04" size="1.27" layer="95" font="vector" rot="R180" xref="yes"/>
-<wire x1="-40.64" y1="66.04" x2="-38.1" y2="66.04" width="0.1524" layer="91"/>
-<pinref part="U$7" gate="G$1" pin="IN1"/>
-</segment>
 <segment>
 <pinref part="BATT_2" gate="G$1" pin="1"/>
@@
 <label x="-220.98" y="-66.04" size="1.27" layer="95" font="vector" xref="yes"/>
 </segment>
+<segment>
+<wire x1="-17.78" y1="60.96" x2="-15.24" y2="60.96" width="0.1524" layer="91"/>
+<label x="-15.24" y="60.96" size="1.27" layer="95" font="vector" xref="yes"/>
+<pinref part="U$7" gate="G$1" pin="IN6"/>
+</segment>
 </net>
 <net name="BATT_EN_1_1" class="0">
@@
 </segment>
 <segment>
-<pinref part="U1" gate="G$1" pin="PB0(ICP)"/>
-<wire x1="17.78" y1="-5.08" x2="22.86" y2="-5.08" width="0.1524" layer="91"/>
-<label x="22.86" y="-5.08" size="1.27" layer="95" font="vector" xref="yes"/>
+<pinref part="U1" gate="G$1" pin="ADC6"/>
+<wire x1="17.78" y1="25.4" x2="22.86" y2="25.4" width="0.1524" layer="91"/>
+<label x="22.86" y="25.4" size="1.27" layer="95" font="vector" xref="yes"/>
 </segment>
 </net>
@@
 <wire x1="-175.26" y1="-68.58" x2="-175.26" y2="-73.66" width="0.1524" layer="91"/>
 <junction x="-175.26" y="-73.66"/>
-</segment>
-</net>
-<net name="BATT_CONN_4" class="0">
-<segment>
-<label x="-15.24" y="58.42" size="1.27" layer="95" font="vector" xref="yes"/>
-<wire x1="-15.24" y1="58.42" x2="-17.78" y2="58.42" width="0.1524" layer="91"/>
-<pinref part="U$7" gate="G$1" pin="IN5"/>
-</segment>
-</net>
-<net name="BATT_CONN_3" class="0">
-<segment>
-<label x="-40.64" y="58.42" size="1.27" layer="95" font="vector" rot="R180" xref="yes"/>
-<wire x1="-40.64" y1="58.42" x2="-38.1" y2="58.42" width="0.1524" layer="91"/>
-<pinref part="U$7" gate="G$1" pin="IN4"/>
 </segment>
 </net>
@@
 <label x="-403.86" y="-66.04" size="1.27" layer="95" font="vector" xref="yes"/>
 </segment>
+<segment>
+<label x="-15.24" y="58.42" size="1.27" layer="95" font="vector" xref="yes"/>
+<wire x1="-15.24" y1="58.42" x2="-17.78" y2="58.42" width="0.1524" layer="91"/>
+<pinref part="U$7" gate="G$1" pin="IN5"/>
+</segment>
 </net>
 <net name="BATT_CONN_1_2" class="0">
@@
 <label x="-403.86" y="-22.86" size="1.27" layer="95" font="vector" xref="yes"/>
 </segment>
-</net>
+<segment>
+<label x="-40.64" y="68.58" size="1.27" layer="95" font="vector" rot="R180" xref="yes"/>
+<wire x1="-40.64" y1="68.58" x2="-38.1" y2="68.58" width="0.1524" layer="91"/>
+<pinref part="U$7" gate="G$1" pin="IN0"/>
+</segment>
+</net>

Commit message: Rerouted ADC Com Lines for Better Analog Lines
Connections:
- net BATT_CONN_1_1: now also U$7.IN6; no longer U$7.IN4
- net BATT_CONN_1_2: now also U$7.IN2; no longer U$7.IN0
- net BATT_CONN_2_1: now also U$7.IN7; no longer U$7.IN6
- net BATT_CONN_2_2: now also U$7.IN3; no longer U$7.IN5
- net CHARGE_SENSE_1: now also U$7.IN1; no longer U$7.IN2
- net CHARGE_SENSE_2: now also U$7.IN0; no longer U$7.IN1
- net I_SENSE_1: now also U$7.IN5; no longer U$7.IN3
- net I_SENSE_2: now also U$7.IN4; no longer U$7.IN7
Changed lines of the file:
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@@
 </segment>
 <segment>
-<label x="-40.64" y="63.5" size="1.27" layer="95" font="vector" rot="R180" xref="yes"/>
-<wire x1="-40.64" y1="63.5" x2="-38.1" y2="63.5" width="0.1524" layer="91"/>
-<pinref part="U$7" gate="G$1" pin="IN2"/>
+<label x="-40.64" y="66.04" size="1.27" layer="95" font="vector" rot="R180" xref="yes"/>
+<wire x1="-40.64" y1="66.04" x2="-38.1" y2="66.04" width="0.1524" layer="91"/>
+<pinref part="U$7" gate="G$1" pin="IN1"/>
 </segment>
 </net>
@@
 </segment>
 <segment>
-<label x="-40.64" y="60.96" size="1.27" layer="95" font="vector" rot="R180" xref="yes"/>
-<wire x1="-40.64" y1="60.96" x2="-38.1" y2="60.96" width="0.1524" layer="91"/>
-<pinref part="U$7" gate="G$1" pin="IN3"/>
+<label x="-15.24" y="58.42" size="1.27" layer="95" font="vector" xref="yes"/>
+<wire x1="-15.24" y1="58.42" x2="-17.78" y2="58.42" width="0.1524" layer="91"/>
+<pinref part="U$7" gate="G$1" pin="IN5"/>
 </segment>
 </net>
@@
 </segment>
 <segment>
-<label x="-40.64" y="66.04" size="1.27" layer="95" font="vector" rot="R180" xref="yes"/>
-<wire x1="-40.64" y1="66.04" x2="-38.1" y2="66.04" width="0.1524" layer="91"/>
-<pinref part="U$7" gate="G$1" pin="IN1"/>
+<label x="-40.64" y="68.58" size="1.27" layer="95" font="vector" rot="R180" xref="yes"/>
+<wire x1="-40.64" y1="68.58" x2="-38.1" y2="68.58" width="0.1524" layer="91"/>
+<pinref part="U$7" gate="G$1" pin="IN0"/>
 </segment>
 </net>
 <net name="I_SENSE_2" class="0">
-<segment>
-<wire x1="-17.78" y1="63.5" x2="-15.24" y2="63.5" width="0.1524" layer="91"/>
-<label x="-15.24" y="63.5" size="1.27" layer="95" font="vector" xref="yes"/>
-<pinref part="U$7" gate="G$1" pin="IN7"/>
-</segment>
 <segment>
 <pinref part="U8" gate="A" pin="OUT"/>
@@
 <wire x1="-340.36" y1="-7.62" x2="-340.36" y2="-5.08" width="0.1524" layer="91"/>
 <junction x="-340.36" y="-5.08"/>
+</segment>
+<segment>
+<label x="-40.64" y="58.42" size="1.27" layer="95" font="vector" rot="R180" xref="yes"/>
+<wire x1="-40.64" y1="58.42" x2="-38.1" y2="58.42" width="0.1524" layer="91"/>
+<pinref part="U$7" gate="G$1" pin="IN4"/>
 </segment>
 </net>
@@
 </segment>
 <segment>
-<label x="-40.64" y="58.42" size="1.27" layer="95" font="vector" rot="R180" xref="yes"/>
-<wire x1="-40.64" y1="58.42" x2="-38.1" y2="58.42" width="0.1524" layer="91"/>
-<pinref part="U$7" gate="G$1" pin="IN4"/>
+<wire x1="-17.78" y1="60.96" x2="-15.24" y2="60.96" width="0.1524" layer="91"/>
+<label x="-15.24" y="60.96" size="1.27" layer="95" font="vector" xref="yes"/>
+<pinref part="U$7" gate="G$1" pin="IN6"/>
 </segment>
 </net>
@@
 </segment>
 <segment>
-<wire x1="-17.78" y1="60.96" x2="-15.24" y2="60.96" width="0.1524" layer="91"/>
-<label x="-15.24" y="60.96" size="1.27" layer="95" font="vector" xref="yes"/>
-<pinref part="U$7" gate="G$1" pin="IN6"/>
+<wire x1="-17.78" y1="63.5" x2="-15.24" y2="63.5" width="0.1524" layer="91"/>
+<label x="-15.24" y="63.5" size="1.27" layer="95" font="vector" xref="yes"/>
+<pinref part="U$7" gate="G$1" pin="IN7"/>
 </segment>
 </net>
@@
 </segment>
 <segment>
-<label x="-15.24" y="58.42" size="1.27" layer="95" font="vector" xref="yes"/>
-<wire x1="-15.24" y1="58.42" x2="-17.78" y2="58.42" width="0.1524" layer="91"/>
-<pinref part="U$7" gate="G$1" pin="IN5"/>
+<label x="-40.64" y="60.96" size="1.27" layer="95" font="vector" rot="R180" xref="yes"/>
+<wire x1="-40.64" y1="60.96" x2="-38.1" y2="60.96" width="0.1524" layer="91"/>
+<pinref part="U$7" gate="G$1" pin="IN3"/>
 </segment>
 </net>
@@
 </segment>
 <segment>
-<label x="-40.64" y="68.58" size="1.27" layer="95" font="vector" rot="R180" xref="yes"/>
-<wire x1="-40.64" y1="68.58" x2="-38.1" y2="68.58" width="0.1524" layer="91"/>
-<pinref part="U$7" gate="G$1" pin="IN0"/>
-</segment>
-</net>
+<label x="-40.64" y="63.5" size="1.27" layer="95" font="vector" rot="R180" xref="yes"/>
+<wire x1="-40.64" y1="63.5" x2="-38.1" y2="63.5" width="0.1524" layer="91"/>
+<pinref part="U$7" gate="G$1" pin="IN2"/>
+</segment>
+</net>
