File: EAGLE Models/Battery Characterizer/Battery Characterizer.sch (EAGLE design)
At the start: 123 parts, among them IC5 FT232RL, Q1 56P2859, T1 IPP80P03P4L04AKSA1, T10 IRLML6401TRPBF, T11 IRLML6401TRPBF, T12 IRLML6401TRPBF, T2 IPP80P03P4L04AKSA1, T3 IPP80P03P4L04AKSA1, T4 IPP80P03P4L04AKSA1, T5 IRF40B207, T6 IRF40B207, T7 STD28P3LLH6AG, T8 STD28P3LLH6AG, T9 IRLML6401TRPBF, U1 ATMEGA328P, U10 MIC4416YM4-TR, U2 INA199A1DCKR, U3 INA199A1DCKR, U4 MIC4416YM4-TR, U5 KA378R05TU, U6 ADR5045AKSZ-REEL7, U8 INA199A1DCKR, U9 INA199A1DCKR, X1 MINI-USB-UX60-MB-5S8

Commit message: Routed Power and Analog in traces, just need enable pins now
Connections:
- net BATT_EN_2_1: now also U1.PD7(AIN1); no longer U1.PD6(AIN0)
- net CHARGE_2_1: now also U1.PD6(AIN0); no longer U1.PD5(T1)
- net DISC_EN_1: now also U1.PD5(T1); no longer U1.PD7(AIN1)
Changed lines of the file:
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@@
 </segment>
 <segment>
-<pinref part="U1" gate="G$1" pin="PD7(AIN1)"/>
-<wire x1="17.78" y1="0" x2="22.86" y2="0" width="0.1524" layer="91"/>
-<label x="22.86" y="0" size="1.27" layer="95" font="vector" xref="yes"/>
+<pinref part="U1" gate="G$1" pin="PD5(T1)"/>
+<wire x1="17.78" y1="5.08" x2="22.86" y2="5.08" width="0.1524" layer="91"/>
+<label x="22.86" y="5.08" size="1.27" layer="95" font="vector" xref="yes"/>
 </segment>
 </net>
@@
 </segment>
 <segment>
-<pinref part="U1" gate="G$1" pin="PD6(AIN0)"/>
-<wire x1="17.78" y1="2.54" x2="22.86" y2="2.54" width="0.1524" layer="91"/>
-<label x="22.86" y="2.54" size="1.27" layer="95" font="vector" xref="yes"/>
+<pinref part="U1" gate="G$1" pin="PD7(AIN1)"/>
+<wire x1="17.78" y1="0" x2="22.86" y2="0" width="0.1524" layer="91"/>
+<label x="22.86" y="0" size="1.27" layer="95" font="vector" xref="yes"/>
 </segment>
 </net>
@@
 </segment>
 <segment>
-<pinref part="U1" gate="G$1" pin="PD5(T1)"/>
-<wire x1="17.78" y1="5.08" x2="22.86" y2="5.08" width="0.1524" layer="91"/>
-<label x="22.86" y="5.08" size="1.27" layer="95" font="vector" xref="yes"/>
-</segment>
-</net>
+<pinref part="U1" gate="G$1" pin="PD6(AIN0)"/>
+<wire x1="17.78" y1="2.54" x2="22.86" y2="2.54" width="0.1524" layer="91"/>
+<label x="22.86" y="2.54" size="1.27" layer="95" font="vector" xref="yes"/>
+</segment>
+</net>

Commit message: Completed First Revision of Battery Characterizer
Parts:
- removed R13, R28: 2.2k, resistor:R-US_R0603
- removed R15, R27: 18k, resistor:R-US_R0603
Connections:
- removed net CHARGE_REF_1: R13.1, R15.2, U3.REF
- removed net CHARGE_REF_2: R27.2, R28.1, U9.REF
- net BATT_CONN_1_1: now also U$7.IN5; no longer U$7.IN6
- net BATT_CONN_1_2: now also U$7.IN1; no longer U$7.IN2
- net BATT_CONN_2_1: now also U$7.IN6; no longer U$7.IN7
- net BATT_CONN_2_2: now also U$7.IN2; no longer U$7.IN3
- net BATT_EN_2_2: now also U1.PC0(ADC0); no longer U1.PC1(ADC1)
- net CHARGE_2_2: now also U1.ADC7; no longer U1.PC0(ADC0)
- net CHARGE_SENSE_1: now also U$7.IN7; no longer U$7.IN1
- net DISC_EN_2: now also U1.PC1(ADC1); no longer U1.ADC7
- net GND: now also U3.REF, U9.REF; no longer R13.2, R28.2
- net I_SENSE_1: now also U$7.IN3; no longer U$7.IN5
- net VCC: no longer R15.1, R27.1
Other:
- note removed: "0.54455 offset"
