File: EAGLE Models/BSPD/BSPD 4 - Copy.brd (EAGLE design)
At the start: 56.8 x 53.3 mm, 32 parts, among them IC1 LT1236S-5

Commit message: Changed resistor values
Changed resistor values
Parts:
- R10: value 1.8k -> 5k
- R7: value 8.2k -> 9.1k
- R8: value 2.2k -> 6.65k
- R9: value 8.87k -> 9.1k
Changed lines of the file:
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@@
 </element>
 <element name="R1" library="SparkFun-Resistors" package="0603-RES" value="1k" x="26.67" y="43.18" rot="R90"/>
-<element name="R10" library="SparkFun-Resistors" package="0603-RES" value="1.8k" x="41.91" y="38.1" rot="R90"/>
+<element name="R10" library="SparkFun-Resistors" package="0603-RES" value="5k" x="41.91" y="38.1" rot="R90"/>
 <element name="R11" library="SparkFun-Resistors" package="0603-RES" value="10k" x="24.13" y="22.86" rot="R90"/>
 <element name="R12" library="SparkFun-Resistors" package="0603-RES" value="10k" x="25.4" y="17.78" rot="R90"/>
@@
 <element name="R5" library="SparkFun-Resistors" package="0603-RES" value="3.3k" x="34.29" y="43.18" rot="R90"/>
 <element name="R6" library="SparkFun-Resistors" package="0603-RES" value="4.7k" x="34.29" y="38.1" rot="R90"/>
-<element name="R7" library="SparkFun-Resistors" package="0603-RES" value="8.2k" x="38.1" y="43.18" rot="R90"/>
-<element name="R8" library="SparkFun-Resistors" package="0603-RES" value="2.2k" x="38.1" y="38.1" rot="R90"/>
-<element name="R9" library="SparkFun-Resistors" package="0603-RES" value="8.87k" x="41.91" y="43.18" rot="R90"/>
+<element name="R7" library="SparkFun-Resistors" package="0603-RES" value="9.1k" x="38.1" y="43.18" rot="R90"/>
+<element name="R8" library="SparkFun-Resistors" package="0603-RES" value="6.65k" x="38.1" y="38.1" rot="R90"/>
+<element name="R9" library="SparkFun-Resistors" package="0603-RES" value="9.1k" x="41.91" y="43.18" rot="R90"/>
 <element name="U$1" library="linear-technology" package="SOIC8" value="LT1018" x="31.75" y="29.21" smashed="yes" rot="R270">
 <attribute name="VALUE" x="28.575" y="31.9405" size="1.27" layer="27"/>

Commit message: Changed resistor value
Changed resistor value
Parts:
- R10: value 5k -> 5.1k
Changed lines of the file:
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@@
 </element>
 <element name="R1" library="SparkFun-Resistors" package="0603-RES" value="1k" x="26.67" y="43.18" rot="R90"/>
-<element name="R10" library="SparkFun-Resistors" package="0603-RES" value="5k" x="41.91" y="38.1" rot="R90"/>
+<element name="R10" library="SparkFun-Resistors" package="0603-RES" value="5.1k" x="41.91" y="38.1" rot="R90"/>
 <element name="R11" library="SparkFun-Resistors" package="0603-RES" value="10k" x="24.13" y="22.86" rot="R90"/>
 <element name="R12" library="SparkFun-Resistors" package="0603-RES" value="10k" x="25.4" y="17.78" rot="R90"/>
