File: EAGLE Models/BSPD/BSPD 4.sch (EAGLE design)
At the start: 32 parts, among them IC1 LT1236S-5

Commit message: added net names for the bspd
Connections:
- net N$16 renamed GND_UNFUSED
- net N$17 renamed 12V_UNFUSED
- net N$18 renamed CURRENT_UNFUSED
- net N$19 renamed BF_UNFUSED
- net N$20 renamed BR_UNFUSED
Changed lines of the file:
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@@
 <?xml version="1.0" encoding="utf-8"?>
 <!DOCTYPE eagle SYSTEM "eagle.dtd">
-<eagle version="7.1.0">
+<eagle version="8.0.1">
 <drawing>
 <settings>
@@
 </segment>
 </net>
-<net name="N$16" class="0">
+<net name="GND_UNFUSED" class="0">
 <segment>
 <pinref part="CONN" gate="G$1" pin="1"/>
@@
 </segment>
 </net>
-<net name="N$17" class="0">
+<net name="12V_UNFUSED" class="0">
 <segment>
 <pinref part="CONN" gate="G$1" pin="2"/>
@@
 </segment>
 </net>
-<net name="N$18" class="0">
+<net name="CURRENT_UNFUSED" class="0">
 <segment>
 <pinref part="CONN" gate="G$1" pin="3"/>
@@
 </segment>
 </net>
-<net name="N$19" class="0">
+<net name="BF_UNFUSED" class="0">
 <segment>
 <pinref part="CONN" gate="G$1" pin="4"/>
@@
 </segment>
 </net>
-<net name="N$20" class="0">
+<net name="BR_UNFUSED" class="0">
 <segment>
 <pinref part="CONN" gate="G$1" pin="5"/>
